File: motor_driver_m1.kicad_sch (KiCad schematic)
At the start: 32 parts, among them J4 Conn_01x01_Pin, J5 Conn_01x01_Pin, J6 Conn_01x01_Pin, M1 DRV8320SRTVR, Q1 NP80N06D6, Q2 NP80N06D6, Q3 NP80N06D6, Q4 NP80N06D6, Q5 NP80N06D6, Q6 NP80N06D6

Commit message: ...
Parts:
- C21: renamed from C18; footprint easyeda2kicad:C0402 -> easyeda2kicad:C0603
- renumbered C16 to C19, C17 to C20, C19 to C22, C20 to C23, C21 to C24, C22 to C25, C23 to C26, R12 to R10, R13 to R11, R14 to R12, R15 to R13, R16 to R14, R17 to R15, R18 to R16, R19 to R17, R20 to R18, R21 to R19, R22 to R20, R6 to R7, R10 to R8, R11 to R9
Other:
- moved on the sheet: J4, J5, J6

Commit message: ...
Connections:
- net SCLK: no longer names the net of M1.20 (SCLK)
- net SDI: no longer names the net of M1.19 (SDI)
- net SDO: no longer names the net of M1.18 (SDO)
- no-connect marks 0 -> 3
Changed lines of the file:
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@@
 		(color 0 0 0 0)
 	)
+	(no_connect
+		(at 96.52 76.2)
+	)
+	(no_connect
+		(at 96.52 71.12)
+	)
+	(no_connect
+		(at 96.52 73.66)
+	)
 	(wire
 		(pts
@@
 	(wire
 		(pts
-			(xy 96.52 76.2) (xy 109.22 76.2)
-		)
-		(stroke
-			(width 0)
-			(type default)
-		)
-	)
-	(wire
-		(pts
 			(xy 85.09 182.88) (xy 85.09 184.15)
 		)
@@
 	(wire
 		(pts
-			(xy 109.22 71.12) (xy 96.52 71.12)
-		)
-		(stroke
-			(width 0)
-			(type default)
-		)
-	)
-	(wire
-		(pts
 			(xy 40.64 182.88) (xy 40.64 184.15)
 		)
@@
 	(wire
 		(pts
-			(xy 109.22 73.66) (xy 96.52 73.66)
-		)
-		(stroke
-			(width 0)
-			(type default)
-		)
-	)
-	(wire
-		(pts
 			(xy 214.63 73.66) (xy 223.52 73.66)
 		)
@@
 		)
 	)
-	(global_label "SDI"
-		(shape input)
-		(at 109.22 73.66 0)
-		(fields_autoplaced yes)
-		(effects
-			(font
-				(size 1.27 1.27)
-			)
-			(justify left)
-		)
-		(property "Intersheetrefs" "${INTERSHEET_REFS}"
-			(at 115.2895 73.66 0)
-			(effects
-				(font
-					(size 1.27 1.27)
-				)
-				(justify left)
-				(hide yes)
-			)
-		)
-	)
 	(global_label "GLC1"
 		(shape input)
@@
 		)
 	)
-	(global_label "SDO"
-		(shape input)
-		(at 109.22 76.2 0)
-		(fields_autoplaced yes)
-		(effects
-			(font
-				(size 1.27 1.27)
-			)
-			(justify left)
-		)
-		(property "Intersheetrefs" "${INTERSHEET_REFS}"
-			(at 116.0152 76.2 0)
-			(effects
-				(font
-					(size 1.27 1.27)
-				)
-				(justify left)
-				(hide yes)
-			)
-		)
-	)
 	(global_label "SHC1"
 		(shape input)
@@
 			(effects
 				(font
-					(size 1.27 1.27)
-				)
-				(justify left)
-				(hide yes)
-			)
-		)
-	)
-	(global_label "SCLK"
-		(shape input)
-		(at 109.22 71.12 0)
-		(fields_autoplaced yes)
-		(effects
-			(font
-				(size 1.27 1.27)
-			)
-			(justify left)
-		)
-		(property "Intersheetrefs" "${INTERSHEET_REFS}"
-			(at 116.9828 71.12 0)
-			(effects
-				(font

Commit message: ...
Parts:
- added C51: 100nF, easyeda2kicad:C0603, symbol Device:C
Connections:
- net B+: now also C51.1
- net GND: now also C51.2
Changed lines of the file:
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@@
 	(generator_version "9.0")
 	(paper "A4")
+	(text_box "BEMF\n"
+		(exclude_from_sim no)
+		(at 30.48 149.86 0)
+		(size 119.38 43.18)
+		(margins 0.9525 0.9525 0.9525 0.9525)
+		(stroke
+			(width 0)
+			(type solid)
+		)
+		(fill
+			(type none)
+		)
+		(effects
+			(font
+				(size 1.27 1.27)
+			)
+			(justify left top)
+		)
+	)
 	(junction
 		(at 118.11 173.99)
@@
 	(wire
 		(pts
+			(xy 96.52 133.35) (xy 96.52 129.54)
+		)
+		(stroke
+			(width 0)
+			(type default)
+		)
+	)
+	(wire
+		(pts
 			(xy 109.22 48.26) (xy 96.52 48.26)
 		)
@@
 	(wire
 		(pts
+			(xy 96.52 118.11) (xy 96.52 121.92)
+		)
+		(stroke
+			(width 0)
+			(type default)
+		)
+	)
+	(wire
+		(pts
 			(xy 85.09 182.88) (xy 85.09 184.15)
 		)
@@
 		)
 	)
+	(global_label "B+"
+		(shape input)
+		(at 96.52 118.11 180)
+		(fields_autoplaced yes)
+		(effects
+			(font
+				(size 1.27 1.27)
+			)
+			(justify right)
+		)
+		(property "Intersheetrefs" "${INTERSHEET_REFS}"
+			(at 90.6924 118.11 0)
+			(effects
+				(font
+					(size 1.27 1.27)
+				)
+				(justify right)
+				(hide yes)
+			)
+		)
+	)
 	(global_label "SHB1"
 		(shape input)
@@
 	)
 	(symbol
+		(lib_id "power:GND")
+		(at 96.52 133.35 0)
+		(unit 1)
+		(exclude_from_sim no)
+		(in_bom yes)
+		(on_board yes)
+		(dnp no)
+		(property "Reference" "#PWR0122"
+			(at 96.52 139.7 0)
+			(effects
+				(font
+					(size 1.27 1.27)
+				)
+				(hide yes)
+			)
+		)
+		(property "Value" "GND"
+			(at 98.552 138.176 0)
+			(effects
+				(font
+					(size 1.27 1.27)
+				)
+				(justify right)
+			)
+		)
+		(property "Footprint" ""
+			(at 96.52 133.35 0)
+			(effects
+				(font
+					(size 1.27 1.27)
+				)
+				(hide yes)
+			)
+		)
+		(property "Datasheet" ""
+			(at 96.52 133.35 0)
+			(effects
+				(font
+					(size 1.27 1.27)
+				)
+				(hide yes)
+			)
+		)
+		(property "Description" "Power symbol creates a global label with name \"GND\" , ground"
+			(at 96.52 133.35 0)
+			(effects
+				(font
+					(size 1.27 1.27)
+				)
+				(hide yes)
+			)
+		)
+		(pin "1"
+		)
+		(instances
+			(project "esc"
+				(path "/131092d7-5dad-4272-a758-a2445b6ec99c/63f0bd9c-70c2-4847-814d-8da099671243"
+					(reference "#PWR0122")
+					(unit 1)
+				)
+			)
+		)
+	)
+	(symbol
 		(lib_id "Connector:Conn_01x01_Pin")
 		(at 43.18 128.27 0)
@@
 					(unit 1)
 				)
+			)
+		)
+	)
+	(symbol
+		(lib_id "Device:C")
+		(at 96.52 125.73 0)
+		(unit 1)
+		(exclude_from_sim no)
+		(in_bom yes)
+		(on_board yes)
+		(dnp no)
+		(property "Reference" "C51"
+			(at 99.314 124.968 0)
+			(effects
+				(font
+					(size 1.27 1.27)
+				)
+				(justify left)
+			)
+		)
+		(property "Value" "100nF"
+			(at 99.314 126.746 0)
+			(effects
+				(font
+					(size 1.27 1.27)
+				)
+				(justify left)
+			)
+		)
+		(property "Footprint" "easyeda2kicad:C0603"
+			(at 97.4852 129.54 0)
+			(effects
+				(font
+					(size 1.27 1.27)
+				)
+				(hide yes)
+			)
+		)
+		(property "Datasheet" "~"
+			(at 96.52 125.73 0)
+			(effects
+				(font
+					(size 1.27 1.27)
+				)
+				(hide yes)
+			)
+		)
+		(property "Description" "Unpolarized capacitor"
+			(at 96.52 125.73 0)
+			(effects
+				(font
+					(size 1.27 1.27)
+				)
+				(hide yes)
+			)
+		)
+		(pin "1"
+		)
+		(pin "2"
+		)
+		(instances
+			(project "esc"
+				(path "/131092d7-5dad-4272-a758-a2445b6ec99c/63f0bd9c-70c2-4847-814d-8da099671243"
+					(reference "C51")
+					(unit 1)
+				)
