File: motor_driver_m1.kicad_sch (KiCad schematic)
At the start: 52 parts, among them J1 Conn_01x01_Pin, J2 Conn_01x01_Pin, J3 Conn_01x01_Pin, M1 STM32C011F6U6TR, Q1 NP80N06D6, Q2 NP80N06D6, Q3 NP80N06D6, Q4 NP80N06D6, Q5 NP80N06D6, Q6 NP80N06D6

Commit message: ...
Parts:
- C10, C11, C12: footprint easyeda2kicad:C0603 -> easyeda2kicad:C1206
Changed lines of the file:
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@@
 			)
 		)
-		(property "Footprint" "easyeda2kicad:C0603"
+		(property "Footprint" "easyeda2kicad:C1206"
 			(at 268.9352 143.51 0)
 			(hide yes)
@@
 			)
 		)
-		(property "Footprint" "easyeda2kicad:C0603"
+		(property "Footprint" "easyeda2kicad:C1206"
 			(at 268.9352 93.98 0)
 			(hide yes)
@@
 			)
 		)
-		(property "Footprint" "easyeda2kicad:C0603"
+		(property "Footprint" "easyeda2kicad:C1206"
 			(at 268.9352 45.72 0)
 			(hide yes)
