File: mcu.kicad_sch (KiCad schematic)
At the start: 24 parts, among them J2 Conn_01x04_Pin, J3 Conn_01x02, U2 STM32F405RGT6, X1 8MHz

Commit message: ...
Parts:
- J2: footprint (none) -> easyeda2kicad:C0603
- J3: footprint (none) -> easyeda2kicad:C0402
- renumbered C7 to C10, C8 to C11, C9 to C12, C10 to C13, C11 to C14, C12 to C15, C13 to C16, C14 to C17, C15 to C18, COSC_IN1 to C6, COSC_OUT1 to C7, C5 to C8, C6 to C9, R60 to R3, R3 to R4, R4 to R5, R5 to R6
Connections:
- net INHA_M3: now also U2.41 (PA8); no longer U2.22 (PA6), U2.43 (PA10)
- net INHB_M3: no longer U2.23 (PA7)
- net INHC_M3: now also U2.43 (PA10); no longer U2.41 (PA8)
- net PHASE_A_M1: now also U2.39 (PC8)
- net PHASE_B_M1: now also U2.38 (PC7)
- net PHASE_C_M1: now also U2.40 (PC9)

Commit message: ...
Parts:
- removed J2: Conn_01x04_Pin, easyeda2kicad:C0603, symbol Connector:Conn_01x04_Pin
- added J2: Conn_01x01_Pin, deshan:Conn_1x1_small, symbol Connector:Conn_01x01_Pin
- J3: footprint easyeda2kicad:C0402 -> (none)
Connections:
- net PWM_M3 is gone; now on net SDO: U2.56 (PB4(NJTRST))
- net PWM_M4 is gone; now on net PHASE_C_M2: U2.57 (PB5)
- net 3V3: now also U2.1 (VBAT)
- net CS_M2: now also U2.2 (PC13); no longer U2.52 (PC11)
- net CS_M4: now also U2.17 (PA3); no longer U2.53 (PC12)
- net EN_M2: now also U2.3 (PC14-OSC32_IN(PC14)); no longer U2.29 (PB10)
- net EN_M4: now also U2.11 (PC3); no longer U2.62 (PB9)
- net INHA_M4: now also U2.16 (PA2); no longer U2.58 (PB6), U2.8 (PC0)
- net INHB_M4: now also U2.15 (PA1); no longer U2.59 (PB7), U2.9 (PC1)
- net INHC_M4: now also U2.14 (PA0-WKUP(PA0)); no longer U2.10 (PC2), U2.61 (PB8)
- net PHASE_A_M2: now also U2.58 (PB6)
- net PHASE_A_M3: now also U2.52 (PC11)
- net PHASE_A_M4: now also U2.20 (PA4); no longer U2.14 (PA0-WKUP(PA0))
- net PHASE_B_M2: now also U2.59 (PB7)
- net PHASE_B_M3: now also U2.54 (PD2)
- net PHASE_B_M4: now also U2.21 (PA5); no longer U2.15 (PA1)
- net PHASE_C_M3: now also U2.53 (PC12)
- net PHASE_C_M4: now also U2.22 (PA6); no longer U2.16 (PA2)
- net SDI: now reaches U2.23 (PA7)
- net DShot: now reaches U2.26 (PB0)
- net DShot: now also J2.1 (Pin_1)
- net PWM_M1: no longer names the net of U2.28 (PB2-BOOT1(PB2))
- net PWM_M2 renamed SCLK
- new net INHA_M2: U2.9 (PC1)
- new net INHB_M2: U2.8 (PC0)
- new net INHC_M2: U2.10 (PC2)
- no-connect marks 8 -> 11
Other:
- moved on the sheet: C6, C7, R3, X1

Commit message: complete change in architecture,work in progress
Parts:
- removed C10, C12, C13, C14, C15, C18: 100nF, easyeda2kicad:C0402, symbol Device:C
- removed C11: 4.7uF, easyeda2kicad:C0603, symbol Device:C
- removed C16: 1uF, easyeda2kicad:C0603, symbol Device:C
- removed C17: 0.1uF, easyeda2kicad:C0603, symbol Device:C
- removed C6, C7: 5pF-25pF, easyeda2kicad:C0402, symbol Device:C
- removed C8, C9: 2.2uF, easyeda2kicad:C0402, symbol Device:C
- removed J2: Conn_01x01_Pin, deshan:Conn_1x1_small, symbol Connector:Conn_01x01_Pin
- removed R3: 10k, easyeda2kicad:R0402, symbol Device:R
- removed R4: 10K, easyeda2kicad:R0402, symbol Device:R
- removed R5, R6: 5K1, easyeda2kicad:R0402, symbol Device:R
- removed U2: STM32F405RGT6, easyeda2kicad:LQFP-64_L10.0-W10.0-P0.50-LS12.0-BL, symbol easyeda2kicad:STM32F405RGT6
- removed USBC1: TYPE-C-31-M-12, easyeda2kicad:USB-C_SMD-TYPE-C-31-M-12_1, symbol easyeda2kicad:TYPE-C-31-M-12
- removed X1: 8MHz, easyeda2kicad:OSC-SMD_3P-L3.2-W1.3-P1.20, symbol easyeda2kicad:CSTNE8M00G520000R0
- removed boot1, reset1: TS-1088-AR02016, easyeda2kicad:SW-SMD_L3.9-W3.0-P4.45, symbol easyeda2kicad:TS-1088-AR02016
Connections:
- no-connect marks 11 -> 0
Other:
- moved on the sheet: J3
