File: esc.kicad_pcb (KiCad board)
At the start: 6 copper layers, 40 x 50 mm, 163 parts, among them J1 Conn_01x02, J10 Conn_01x01_Pin, J11 Conn_01x01_Pin, J12 Conn_01x01_Pin, J13 Conn_01x01_Pin, J14 Conn_01x01_Pin, J15 Conn_01x01_Pin, J4 Conn_01x01_Pin, J5 Conn_01x01_Pin, J6 Conn_01x01_Pin, J7 Conn_01x01_Pin, J8 Conn_01x01_Pin, J9 Conn_01x01_Pin, M1 DRV8320SRTVR, M2 DRV8320SRTVR, M3 DRV8320SRTVR, M4 DRV8320SRTVR, Q1 NP80N06D6, Q10 NP80N06D6, Q11 NP80N06D6, Q12 NP80N06D6, Q13 NP80N06D6, Q14 NP80N06D6, Q15 NP80N06D6, Q16 NP80N06D6, Q17 NP80N06D6, Q18 NP80N06D6, Q19 NP80N06D6, Q2 NP80N06D6, Q20 NP80N06D6, Q21 NP80N06D6, Q22 NP80N06D6, Q23 NP80N06D6, Q24 NP80N06D6, Q3 NP80N06D6, Q4 NP80N06D6, Q5 NP80N06D6, Q6 NP80N06D6, Q7 NP80N06D6, Q8 NP80N06D6, Q9 NP80N06D6, U1 AP63201WU-7, U2 STM32F405RGT6, X1 8MHz

Commit message: ...
Parts:
- removed C2.1, C2.2: 22uF, easyeda2kicad:C0603
- removed COSC_IN1, COSC_OUT1: 5pF-25pF, easyeda2kicad:C0402
- removed R35, R62, R63, R64, R65, R66, R67, R69, R71, R73: 10k, easyeda2kicad:R0402
- removed R68, R70, R72: 100k, easyeda2kicad:R0402
- added C0: 470uF, easyeda2kicad:CAP-TH_BD10.0-P5.00-D0.6-FD_1, F.Cu at (230.0, 83.0)
- added C48: 4.7nF, easyeda2kicad:C0402, F.Cu at (254.9, 29.5)
- added C49: 4.7nF, easyeda2kicad:C0402, F.Cu at (255.4, 27.2)
- added C50: 4.7nF, easyeda2kicad:C0402, F.Cu at (259.0, 74.0)
- added J2: Conn_01x04_Pin, easyeda2kicad:C0603, F.Cu at (1.44, 0.76)
- added J3: Conn_01x02, easyeda2kicad:C0402, F.Cu at (0.92, 3.07)
- added R24: 10k, easyeda2kicad:R0402, F.Cu at (250.1, 24.3)
- added R25: 10k, easyeda2kicad:R0402, F.Cu at (250.1, 26.4)
- added R26: 10k, easyeda2kicad:R0402, F.Cu at (250.1, 28.5)
- added R40: 10k, easyeda2kicad:R0402, F.Cu at (245.1, 16.0)
- added R41: 10k, easyeda2kicad:R0402, F.Cu at (245.1, 18.1)
- added R42: 10k, easyeda2kicad:R0402, F.Cu at (245.1, 20.2)
- added R43: 100k, easyeda2kicad:R0402, F.Cu at (245.1, 22.3)
- added R57: 10k, easyeda2kicad:R0402, F.Cu at (255.1, 16.0)
- added R58: 100k, easyeda2kicad:R0402, F.Cu at (255.1, 18.1)
- added R59: 10k, easyeda2kicad:R0402, F.Cu at (255.1, 20.2)
- added R7: 10k, easyeda2kicad:R0402, B.Cu at (230.5, 43.5)
- added R8: 10k, easyeda2kicad:R0402, F.Cu at (237.4, 42.3)
- added R9: 10k, easyeda2kicad:R0402, F.Cu at (248.0, 55.3)
- C10, R10: moved to B.Cu
- C11: value 100nF -> 4.7uF; footprint easyeda2kicad:C0402 -> easyeda2kicad:C0603
- C13: value 1uF -> 100nF; footprint easyeda2kicad:C0603 -> easyeda2kicad:C0402
- C14: value 0.1uF -> 100nF; footprint easyeda2kicad:C0603 -> easyeda2kicad:C0402
- C16: value >10uF -> 1uF
- C17: footprint easyeda2kicad:C0402 -> easyeda2kicad:C0603
- C18: value 1uF -> 100nF
- C19: value 47nF -> >10uF; moved to B.Cu
- C2: value 470uF -> 100nF; footprint easyeda2kicad:CAP-TH_BD10.0-P5.00-D0.6-FD_1 -> easyeda2kicad:C0603
- C20: value 1uF -> 0.1uF; footprint easyeda2kicad:C0603 -> easyeda2kicad:C0402; moved to B.Cu
- C21, C29, C31, C37, C39, C45, C47: value 4.7nF -> 1uF; footprint easyeda2kicad:C0402 -> easyeda2kicad:C0603
- C22: value 4.7nF -> 47nF; footprint easyeda2kicad:C0402 -> easyeda2kicad:C0603; moved to F.Cu
- C23: value 4.7nF -> 1uF; footprint easyeda2kicad:C0402 -> easyeda2kicad:C0603; moved to F.Cu
- C24: value >10uF -> 4.7nF; footprint easyeda2kicad:C0603 -> easyeda2kicad:C0402; moved to B.Cu
- C25: value 0.1uF -> 4.7nF; footprint easyeda2kicad:C0603 -> easyeda2kicad:C0402; moved to B.Cu
- C26: value 1uF -> 4.7nF; footprint easyeda2kicad:C0603 -> easyeda2kicad:C0402; moved to B.Cu
- C27, C35, C43: value 47nF -> >10uF
- C28, C36: value 1uF -> 0.1uF; footprint easyeda2kicad:C0603 -> easyeda2kicad:C0402
- C3: value 100nF -> 100pF
- C30, C38, C46: value 4.7nF -> 47nF; footprint easyeda2kicad:C0402 -> easyeda2kicad:C0603
- C32, C40: value >10uF -> 4.7nF; footprint easyeda2kicad:C0603 -> easyeda2kicad:C0402; moved to F.Cu
- C33, C41: value 0.1uF -> 4.7nF; footprint easyeda2kicad:C0603 -> easyeda2kicad:C0402; moved to F.Cu
- C34, C42: value 1uF -> 4.7nF; footprint easyeda2kicad:C0603 -> easyeda2kicad:C0402; moved to F.Cu
- C4: value 100pF -> 22uF
- C44: value 1uF -> 0.1uF; footprint easyeda2kicad:C0603 -> easyeda2kicad:C0402; moved to F.Cu
- C5: value 2.2uF -> 22uF; footprint easyeda2kicad:C0402 -> easyeda2kicad:C0603
- C6: value 2.2uF -> 5pF-25pF; moved to B.Cu
- C7: value 100nF -> 5pF-25pF
- C8: value 4.7uF -> 2.2uF; footprint easyeda2kicad:C0603 -> easyeda2kicad:C0402
- C9: value 100nF -> 2.2uF
- R1: value 196K -> 62K; footprint easyeda2kicad:R0805 -> easyeda2kicad:R0603
- R15: value 10k -> 100k; moved to B.Cu
- R2: value 62K -> 196K; footprint easyeda2kicad:R0603 -> easyeda2kicad:R0805
- R21, R34, R36, R38, R51, R53, R55: value 100k -> 10k
- R29, R31, R33, R45, R47, R56, R60: value 10k -> 100k
- R3: value 10K -> 10k
- R4: value 5K1 -> 10K
- R6: value 10k -> 5K1
- R61: moved to F.Cu
- moved J7 81.5 mm to (206.8, 65.2)
- moved J8 81.5 mm to (206.8, 69.2)
- moved J9 81.5 mm to (206.8, 73.2)
- moved J12 54.6 mm to (211.6, 56.4), turned to 180 degrees
- moved J11 54.2 mm to (211.6, 50.9), turned to 180 degrees
- moved J10 53.9 mm to (211.6, 45.4), turned to 180 degrees
- moved C26 51.1 mm to (234.1, 45.5), turned to 180 degrees
- moved C25 50.2 mm to (235.5, 47.1), turned to 90 degrees
- moved C24 45.6 mm to (234.7, 54.3), turned to -90 degrees
- moved C32 45.4 mm to (271.7, 46.0)
- moved C33 44.9 mm to (271.7, 48.5)
- moved C35 44.7 mm to (186.4, 64.9)
- moved C34 44.6 mm to (271.7, 51.0), turned to 0 degrees
- moved C44 42.1 mm to (271.7, 63.1)
- moved C42 39.3 mm to (271.7, 60.6), turned to 0 degrees
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Connections:
- C12 pad 1: 3V3 -> GND
- C12 pad 2: GND -> 3V3
- C13 pad 1: 3V3 -> GND
- C13 pad 2: GND -> 3V3
- C14 pad 1: RESET -> GND
- C14 pad 2: GND -> 3V3
- C15 pad 1: BOOT0 -> 3V3
- C16 pad 1: B+ -> 3V3
- C17 pad 1: B+ -> RESET
- C18 pad 1: B+ -> BOOT0
- C18 pad 2: Net-(M1-VCP) -> GND
- C19 pad 1: Net-(M1-CPL) -> B+
- C19 pad 2: Net-(M1-CPH) -> GND
- C2 pad 1: GND -> Net-(U1-BST)
- C2 pad 2: B+ -> Net-(U1-SW)
- C20 pad 1: Net-(M1-DVDD) -> B+
- C21 pad 1: PHASE_A_M1 -> B+
- C21 pad 2: GND -> Net-(M1-VCP)
- C22 pad 1: PHASE_B_M1 -> Net-(M1-CPL)
- C22 pad 2: GND -> Net-(M1-CPH)
- C23 pad 1: PHASE_C_M1 -> Net-(M1-DVDD)
- C24 pad 1: B+ -> PHASE_A_M1
- C25 pad 1: B+ -> PHASE_B_M1
- C26 pad 1: B+ -> PHASE_C_M1
- C26 pad 2: Net-(M2-VCP) -> GND
- C27 pad 1: Net-(M2-CPL) -> B+
- C27 pad 2: Net-(M2-CPH) -> GND
- C28 pad 1: Net-(M2-DVDD) -> B+
- C29 pad 1: PHASE_A_M2 -> B+
- C29 pad 2: GND -> Net-(M2-VCP)
- C3 pad 1: Net-(U1-BST) -> Net-(U1-FB)
- C3 pad 2: Net-(U1-SW) -> 3V3
- C30 pad 1: PHASE_B_M2 -> Net-(M2-CPL)
- C30 pad 2: GND -> Net-(M2-CPH)
- C31 pad 1: PHASE_C_M2 -> Net-(M2-DVDD)
- C32 pad 1: B+ -> PHASE_A_M2
- C33 pad 1: B+ -> PHASE_B_M2
- C34 pad 1: B+ -> PHASE_C_M2
- C34 pad 2: Net-(M3-VCP) -> GND
- C35 pad 1: Net-(M3-CPL) -> B+
- C35 pad 2: Net-(M3-CPH) -> GND
- C36 pad 1: Net-(M3-DVDD) -> B+
- C37 pad 1: PHASE_A_M3 -> B+
- C37 pad 2: GND -> Net-(M3-VCP)
- C38 pad 1: PHASE_B_M3 -> Net-(M3-CPL)
- C38 pad 2: GND -> Net-(M3-CPH)
- C39 pad 1: PHASE_C_M3 -> Net-(M3-DVDD)
- C4 pad 1: Net-(U1-FB) -> 3V3
- C4 pad 2: 3V3 -> GND
- C40 pad 1: B+ -> PHASE_A_M3
- C41 pad 1: B+ -> PHASE_B_M3
- C42 pad 1: B+ -> PHASE_C_M3
- C42 pad 2: Net-(M4-VCP) -> GND
- C43 pad 1: Net-(M4-CPL) -> B+
- C43 pad 2: Net-(M4-CPH) -> GND
- C44 pad 1: Net-(M4-DVDD) -> B+
- C45 pad 1: PHASE_A_M4 -> B+
- C45 pad 2: GND -> Net-(M4-VCP)
- C46 pad 1: PHASE_B_M4 -> Net-(M4-CPL)
- C46 pad 2: GND -> Net-(M4-CPH)
- C47 pad 1: PHASE_C_M4 -> Net-(M4-DVDD)
- C5 pad 1: GND -> 3V3
- C5 pad 2: Net-(U2A-VCAP_1) -> GND
- C6 pad 1: GND -> Net-(U2A-PH0-OSC_IN(PH0))
- C6 pad 2: Net-(U2A-VCAP_2) -> GND
- C7 pad 2: 3V3 -> Net-(U2A-PH1-OSC_OUT(PH1))
- C8 pad 2: 3V3 -> Net-(U2A-VCAP_1)
- C9 pad 2: 3V3 -> Net-(U2A-VCAP_2)
- J10 pad 1: SHC3 -> SHA3
- J11 pad 1: SHA3 -> SHB3
- J12 pad 1: SHB3 -> SHC3
- J13 pad 1: SHC4 -> SHA4
- J14 pad 1: SHA4 -> SHB4
- J15 pad 1: SHB4 -> SHC4
- J7 pad 1: SHC2 -> SHA2
- J8 pad 1: SHA2 -> SHB2
- J9 pad 1: SHB2 -> SHC2
- R1 pad 1: 3V3 -> Net-(U1-FB)
- R1 pad 2: Net-(U1-FB) -> GND
- R10 pad 1: Net-(M1-nFAULT) -> GLA1
- R10 pad 2: 3V3 -> GND
- R11 pad 1: GHA1 -> GHB1
- R11 pad 2: SHA1 -> SHB1
- R12 pad 1: GLA1 -> GLB1
- R13 pad 1: GHB1 -> GHC1
- R13 pad 2: SHB1 -> SHC1
- R14 pad 1: GLB1 -> GLC1
- R15 pad 1: GHC1 -> PHASE_A_M1
- R15 pad 2: SHC1 -> SHA1
- R16 pad 1: GLC1 -> GND
- R16 pad 2: GND -> PHASE_A_M1
- R17 pad 1: PHASE_A_M1 -> PHASE_B_M1
- R17 pad 2: SHA1 -> SHB1
- R18 pad 2: PHASE_A_M1 -> PHASE_B_M1
- R19 pad 1: PHASE_B_M1 -> PHASE_C_M1
- R19 pad 2: SHB1 -> SHC1
- R2 pad 1: Net-(U1-FB) -> 3V3
- R2 pad 2: GND -> Net-(U1-FB)
- R20 pad 2: PHASE_B_M1 -> PHASE_C_M1
- R21 pad 1: PHASE_C_M1 -> 3V3
- R21 pad 2: SHC1 -> PUPL2
- R22 pad 1: GND -> Net-(M2-nFAULT)
- R22 pad 2: PHASE_C_M1 -> 3V3
- R23 pad 1: 3V3 -> GHA2
- R23 pad 2: PUPL2 -> SHA2
- R27 pad 1: Net-(M2-nFAULT) -> GHC2
- R27 pad 2: 3V3 -> SHC2
- R28 pad 1: GHA2 -> GLC2
- R28 pad 2: SHA2 -> GND
- R29 pad 1: GLA2 -> PHASE_A_M2
- R29 pad 2: GND -> SHA2
- R3 pad 1: BOOT0 -> SDO
- R3 pad 2: GND -> 3V3
- R30 pad 1: GHB2 -> GND
- R30 pad 2: SHB2 -> PHASE_A_M2
- R31 pad 1: GLB2 -> PHASE_B_M2
- R31 pad 2: GND -> SHB2
- R32 pad 1: GHC2 -> GND
- R32 pad 2: SHC2 -> PHASE_B_M2
- R33 pad 1: GLC2 -> PHASE_C_M2
- R33 pad 2: GND -> SHC2
- R34 pad 1: PHASE_A_M2 -> GND
- R34 pad 2: SHA2 -> PHASE_C_M2
- R36 pad 1: PHASE_B_M2 -> Net-(M3-nFAULT)
- R36 pad 2: SHB2 -> 3V3
- R37 pad 1: GND -> GHA3
- R37 pad 2: PHASE_B_M2 -> SHA3
- R38 pad 1: PHASE_C_M2 -> GLA3
- R38 pad 2: SHC2 -> GND
- R39 pad 1: GND -> GHB3
- R39 pad 2: PHASE_C_M2 -> SHB3
- R4 pad 1: GND -> BOOT0
- R4 pad 2: Net-(USBC1-CC1) -> GND
- R44 pad 1: Net-(M3-nFAULT) -> GND
- R44 pad 2: 3V3 -> PHASE_A_M3
- R45 pad 1: GHA3 -> PHASE_B_M3
- R45 pad 2: SHA3 -> SHB3
- R46 pad 1: GLA3 -> GND
- R46 pad 2: GND -> PHASE_B_M3
- R47 pad 1: GHB3 -> PHASE_C_M3
- R47 pad 2: SHB3 -> SHC3
- R48 pad 1: GLB3 -> GND
- R48 pad 2: GND -> PHASE_C_M3
- R49 pad 1: GHC3 -> Net-(M4-nFAULT)
- R49 pad 2: SHC3 -> 3V3
- R5 pad 2: Net-(USBC1-CC2) -> Net-(USBC1-CC1)
- R50 pad 1: GLC3 -> GHA4
- R50 pad 2: GND -> SHA4
- R51 pad 1: PHASE_A_M3 -> GLA4
- R51 pad 2: SHA3 -> GND
- R52 pad 1: GND -> GHB4
- R52 pad 2: PHASE_A_M3 -> SHB4
- R53 pad 1: PHASE_B_M3 -> GLB4
- R53 pad 2: SHB3 -> GND
- R54 pad 1: GND -> GHC4
- R54 pad 2: PHASE_B_M3 -> SHC4
- R55 pad 1: PHASE_C_M3 -> GLC4
- R55 pad 2: SHC3 -> GND
- R56 pad 1: GND -> PHASE_A_M4
- R56 pad 2: PHASE_C_M3 -> SHA4
- R6 pad 1: 3V3 -> GND
- R6 pad 2: PUPL1 -> Net-(USBC1-CC2)
- R60 pad 1: SDO -> PHASE_C_M4
- R60 pad 2: 3V3 -> SHC4
- R61 pad 1: Net-(M4-nFAULT) -> GND
- R61 pad 2: 3V3 -> PHASE_C_M4
- U2 pad 22: INHA_M3 -> unconnected-(U2A-PA6-Pad22)
- U2 pad 23: INHB_M3 -> unconnected-(U2A-PA7-Pad23)
- U2 pad 38: unconnected-(U2A-PC7-Pad38) -> PHASE_B_M1
- U2 pad 39: unconnected-(U2A-PC8-Pad39) -> PHASE_A_M1
- U2 pad 40: unconnected-(U2A-PC9-Pad40) -> PHASE_C_M1
- U2 pad 41: INHC_M3 -> INHA_M3
- U2 pad 43: INHA_M3 -> INHC_M3
Routing:
- net GHB3: track 21.0 -> 0.35 mm, vias 2 -> 1
- net D-: track 0.00 -> 19.9 mm, vias 0 -> 2
- net D+: track 0.00 -> 19.8 mm, vias 0 -> 2
- net GHA3: track 19.0 -> 0.10 mm
- net GHC3: track 16.4 -> 0.04 mm, vias 2 -> 1
- net PHASE_C_M1: track 0.00 -> 14.0 mm, vias 0 -> 1
- net PHASE_B_M1: track 0.00 -> 12.8 mm, vias 0 -> 1
- net SHC3: track 10.6 -> 0.00 mm, vias 10 -> 9
- net INHC_M3: track 1.05 -> 10.4 mm, vias 1 -> 2
- net GLA3: track 8.46 -> 0.25 mm
- net PUPL1: track 10.1 -> 18.0 mm
- net PHASE_A_M1: track 0.00 -> 7.53 mm, vias 0 -> 1
- net INHB_M3: track 1.03 -> 7.72 mm, vias 1 -> 2
- net GLA4: track 5.65 -> 0.00 mm
- net INHA_M3: track 1.02 -> 6.35 mm, vias 1 -> 0
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- added copper zone on B.Cu, net GND
- added copper zone on F.Cu, net SHA1
- added copper zone on F.Cu, net SHB1
- added copper zone on F.Cu, net SHC1

Commit message: ...
Parts:
- removed J3: Conn_01x02, easyeda2kicad:C0402
- C10, C11, Q10, Q12, Q14, Q16, Q18, Q8, R22, R3, R50: moved to F.Cu
- C2, C27, C28, C29, C32, C33, C34, C36, C37, C38, C40, C41, C42, C44, C45, C47, C48, C49, C50, Q11, Q13, Q15, Q17, Q7, Q9, R29, R30, R31, R32, R33, R34, R43, R45, R47, R51, R53, R55, R56, R57, R58, R59, R60, R61: moved to B.Cu
- J2: value Conn_01x04_Pin -> Conn_01x01_Pin; footprint easyeda2kicad:C0603 -> deshan:Conn_1x1_small
- moved J2 242.2 mm to (240.2, 41.0), turned to 90 degrees
- moved C5 67.1 mm to (235.1, 94.3), turned to -90 degrees
- moved R57 64.7 mm to (235.5, 77.6), turned to 90 degrees
- moved R59 57.2 mm to (235.5, 73.9), turned to 90 degrees
- moved R58 57.1 mm to (236.5, 72.0), turned to 90 degrees
- moved R25 56.4 mm to (211.1, 67.1), turned to 180 degrees
- moved R54 55.3 mm to (248.0, 61.6), turned to 0 degrees
- moved reset1 54.7 mm to (235.5, 78.4), turned to 180 degrees
- moved R52 54.5 mm to (248.0, 67.1), turned to 0 degrees
- moved R56 54.3 mm to (236.9, 77.2), turned to 0 degrees
- moved boot1 54.0 mm to (224.5, 78.4), turned to 180 degrees
- moved C34 52.9 mm to (224.2, 74.1), turned to 90 degrees
- moved C48 52.2 mm to (234.5, 77.6), turned to -90 degrees
- moved C33 52.0 mm to (225.3, 72.0), turned to -90 degrees
- moved C40 51.9 mm to (221.1, 43.7), turned to 180 degrees
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Connections:
- J2 pad 1: PWM_M1 -> DShot
- M1 pad 18: SDO -> unconnected-(M1-SDO-Pad18)
- M1 pad 19: SDI -> unconnected-(M1-SDI-Pad19)
- M1 pad 20: SCLK -> unconnected-(M1-SCLK-Pad20)
- M2 pad 18: SDO -> unconnected-(M2-SDO-Pad18)
- M2 pad 19: SDI -> unconnected-(M2-SDI-Pad19)
- M2 pad 20: SCLK -> unconnected-(M2-SCLK-Pad20)
- M3 pad 18: SDO -> unconnected-(M3-SDO-Pad18)
- M3 pad 19: SDI -> unconnected-(M3-SDI-Pad19)
- M3 pad 20: SCLK -> unconnected-(M3-SCLK-Pad20)
- M4 pad 18: SDO -> unconnected-(M4-SDO-Pad18)
- M4 pad 19: SDI -> unconnected-(M4-SDI-Pad19)
- M4 pad 20: SCLK -> unconnected-(M4-SCLK-Pad20)
- U2 pad 1: unconnected-(U2B-VBAT-Pad1) -> 3V3
- U2 pad 10: INHC_M4 -> INHC_M2
- U2 pad 11: unconnected-(U2A-PC3-Pad11) -> EN_M4
- U2 pad 14: PHASE_A_M4 -> INHC_M4
- U2 pad 15: PHASE_B_M4 -> INHB_M4
- U2 pad 16: PHASE_C_M4 -> INHA_M4
- U2 pad 17: unconnected-(U2A-PA3-Pad17) -> CS_M4
- U2 pad 2: unconnected-(U2A-PC13-Pad2) -> CS_M2
- U2 pad 20: unconnected-(U2A-PA4-Pad20) -> PHASE_A_M4
- U2 pad 21: unconnected-(U2A-PA5-Pad21) -> PHASE_B_M4
- U2 pad 22: unconnected-(U2A-PA6-Pad22) -> PHASE_C_M4
- U2 pad 23: unconnected-(U2A-PA7-Pad23) -> SDI
- U2 pad 26: unconnected-(U2A-PB0-Pad26) -> DShot
- U2 pad 28: PWM_M1 -> unconnected-(U2A-PB2-BOOT1(PB2)-Pad28)
- U2 pad 29: EN_M2 -> unconnected-(U2A-PB10-Pad29)
- U2 pad 3: unconnected-(U2A-PC14-OSC32_IN(PC14)-Pad3) -> EN_M2
- U2 pad 52: CS_M2 -> PHASE_A_M3
- U2 pad 53: CS_M4 -> PHASE_C_M3
- U2 pad 54: unconnected-(U2A-PD2-Pad54) -> PHASE_B_M3
- U2 pad 55: PWM_M2 -> SCLK
- U2 pad 56: PWM_M3 -> SDO
- U2 pad 57: PWM_M4 -> PHASE_C_M2
- U2 pad 58: INHA_M4 -> PHASE_A_M2
- U2 pad 59: INHB_M4 -> PHASE_B_M2
- U2 pad 61: INHC_M4 -> unconnected-(U2A-PB8-Pad61)
- U2 pad 62: EN_M4 -> unconnected-(U2A-PB9-Pad62)
- U2 pad 8: INHA_M4 -> INHB_M2
- U2 pad 9: INHB_M4 -> INHA_M2
Routing:
- net GND: track 49.9 -> 152.9 mm, vias 68 -> 102
- net BOOT0: track 1.28 -> 34.6 mm, vias 1 -> 2
- net RESET: track 0.00 -> 26.1 mm, vias 0 -> 3
- net SHC4: track 10.3 -> 34.9 mm, vias 10 -> 11
- net PHASE_A_M3: track 0.00 -> 22.0 mm, vias 0 -> 1
- net SHC3: track 0.00 -> 21.7 mm, vias 9 -> 10
- net B+: track 10.5 -> 31.4 mm, vias 46 -> 55
- net GHA2: track 0.00 -> 20.7 mm, vias 0 -> 2
- net GHC3: track 0.04 -> 20.7 mm, vias 1 -> 2
- net PHASE_C_M2: track 0.00 -> 20.5 mm, vias 0 -> 1
- net GHA3: track 0.10 -> 18.6 mm
- net GHB3: track 0.35 -> 18.5 mm, vias 1 -> 2
- net PUPL2: track 0.00 -> 17.7 mm, vias 0 -> 3
- net PHASE_A_M4: track 0.00 -> 17.7 mm, vias 0 -> 1
- net SHA2: track 0.00 -> 17.6 mm, vias 0 -> 10
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- added copper zone on B.Cu, net B+
- added copper zone on B.Cu, net SHA2
- added copper zone on F.Cu, net SHA2
- added copper zone on F.Cu, net SHA3
- added copper zone on B.Cu, net SHA4
- added copper zone on F.Cu, net SHA4
- added copper zone on B.Cu, net SHB2
- added copper zone on F.Cu, net SHB2
- added copper zone on F.Cu, net SHB3
- added copper zone on B.Cu, net SHB4
- added copper zone on F.Cu, net SHB4
- added copper zone on B.Cu, net SHC2
- added copper zone on F.Cu, net SHC2
- added copper zone on F.Cu, net SHC3
- added copper zone on B.Cu, net SHC4
- added copper zone on F.Cu, net SHC4

Commit message: ESC_V1.0
Parts:
- removed C1: 10uF, easyeda2kicad:C1206
- removed C2: 100nF, easyeda2kicad:C0603
- removed C3: 100pF, easyeda2kicad:C0603
- removed C4, C5: 22uF, easyeda2kicad:C0603
- removed L1: 6.8uH, easyeda2kicad:IND-SMD_L2.5-W2.0_FTC252010S
- removed R1: 62K, easyeda2kicad:R0603
- removed R2: 196K, easyeda2kicad:R0805
- removed U1: AP63201WU-7, easyeda2kicad:TSOT-23-6_L2.9-W1.6-P0.95-LS2.8-BR
- added J16: Conn_01x02, deshan:Batt_Conn_HV, B.Cu at (230.0, 83.0)
- added J17: Conn_01x01_Pin, deshan:Conn_1x1_small, F.Cu at (220.0, 41.0)
- moved C44 5.47 mm to (228.6, 76.8), turned to -90 degrees
- moved C43 3.84 mm to (229.8, 76.8), turned to -90 degrees
- moved R39 0.71 mm to (211.8, 49.6)
- moved R23 0.70 mm to (211.8, 61.6)
- moved R25 0.70 mm to (211.8, 67.1)
- moved R27 0.70 mm to (211.8, 72.6)
- moved R41 0.70 mm to (211.8, 55.1)
- moved C45 0.68 mm to (231.2, 76.8)
- moved R37 0.54 mm to (211.6, 44.5)
- moved C22 0.26 mm to (230.5, 50.6)
- moved J2 0.24 mm to (240.0, 41.0)
- moved R11 0.20 mm to (248.0, 49.6)
- moved R9 0.20 mm to (248.0, 55.1)
- moved R13 0.10 mm to (248.0, 44.3)
- moved J1 0.05 mm to (230.0, 83.0)
Routing:
- net GND: track 152.9 -> 187.3 mm, vias 102 -> 109
- net DShot: track 1.02 -> 21.8 mm, vias 1 -> 2
- net B+: track 31.4 -> 36.0 mm, vias 55 -> 54
- net 3V3: track 17.5 -> 21.9 mm, vias 9 -> 12
- net Net-(M4-VCP): track 2.20 -> 3.69 mm
- net SHB3: track 17.0 -> 15.7 mm
- net GHA3: track 18.6 -> 17.3 mm
- net SCLK: track 1.15 -> 0.00 mm, vias 1 -> 0
- net SDO: track 3.02 -> 2.00 mm, vias 1 -> 0
- net GHB3: track 18.5 -> 17.6 mm
- net CS_M2: track 14.6 -> 13.9 mm
- net PHASE_A_M3: track 22.0 -> 21.4 mm
- net GLA3: track 8.20 -> 7.68 mm
- net PHASE_B_M3: track 15.5 -> 15.0 mm

Commit message: edited symbols
Parts:
- moved C35 0.26 mm to (227.8, 47.1)
- moved C19 0.18 mm to (233.1, 47.5)
- moved C27 0.08 mm to (225.5, 69.6)
- moved R31 0.08 mm to (223.3, 71.2)
- moved C15 0.06 mm to (231.9, 64.4)
- moved R32 0.05 mm to (224.3, 72.0)
Routing:
- net GND: track 187.3 -> 188.4 mm
Other:
- board text added: "3V3"
- board text added: "DShot"

Commit message: ...
Parts:
- added C51: 100nF, easyeda2kicad:C0603, F.Cu at (244.0, 41.0)
- added C52: 100nF, easyeda2kicad:C0603, F.Cu at (216.0, 79.0)
- added C53: 100nF, easyeda2kicad:C0603, F.Cu at (216.0, 41.0)
- added C54: 100nF, easyeda2kicad:C0603, F.Cu at (244.0, 79.0)
Routing:
- net GND: vias 109 -> 113

Commit message: complete change in architecture,work in progress
Parts:
- removed M1, M2, M3, M4: DRV8320SRTVR, easyeda2kicad:WQFN-32_L5.0-W5.0-P0.50-TL-EP3.5
- removed USBC1: TYPE-C-31-M-12, easyeda2kicad:USB-C_SMD-TYPE-C-31-M-12_1
- removed X1: 8MHz, easyeda2kicad:OSC-SMD_3P-L3.2-W1.3-P1.20
- removed boot1, reset1: TS-1088-AR02016, easyeda2kicad:SW-SMD_L3.9-W3.0-P4.45
- added C55: 4.7uF, easyeda2kicad:C0402, F.Cu at (231.3, 60.4)
- added C56: 100nF, easyeda2kicad:C0402, F.Cu at (233.6, 59.9)
- added C57: 1uF, easyeda2kicad:C0402, B.Cu at (225.2, 54.1)
- added C58: 100nF, easyeda2kicad:C0603, B.Cu at (236.8, 52.0)
- added C59: 100nF, easyeda2kicad:C0603, B.Cu at (236.8, 57.5)
- added C60: 100nF, easyeda2kicad:C0603, F.Cu at (223.2, 45.4)
- added C61: 100nF, easyeda2kicad:C0603, F.Cu at (223.2, 51.0)
- added C62: 100nF, easyeda2kicad:C0603, B.Cu at (236.8, 69.6)
- added C63: 100nF, easyeda2kicad:C0603, B.Cu at (236.8, 64.1)
- added C64: 100nF, easyeda2kicad:C0603, B.Cu at (223.1, 68.5)
- added C65: 100nF, easyeda2kicad:C0603, B.Cu at (223.1, 73.9)
- added J18: Conn_01x01_Pin, deshan:Conn_1x1_small, F.Cu at (221.9, 79.0)
- added J19: Conn_01x01_Pin, deshan:Conn_1x1_small, F.Cu at (221.8, 41.1)
- added J20: Conn_01x01_Pin, deshan:Conn_1x1_small, F.Cu at (238.4, 78.9)
- added R35: 10k, easyeda2kicad:R0402, F.Cu at (232.3, 44.2)
- added R62: 10k, easyeda2kicad:R0402, F.Cu at (232.0, 77.7)
- added R63: 10k, easyeda2kicad:R0402, F.Cu at (226.6, 63.7)
- added R64: 10k, easyeda2kicad:R0402, F.Cu at (228.0, 65.3)
- added R65: 50k, easyeda2kicad:R0402, F.Cu at (227.1, 65.3)
- added R66: 10k, easyeda2kicad:R0402, B.Cu at (229.0, 77.7)
- added R67: 10k, easyeda2kicad:R0402, B.Cu at (233.6, 63.8)
- added R68: 10k, easyeda2kicad:R0402, B.Cu at (232.2, 65.2)
- added R69: 50k, easyeda2kicad:R0402, B.Cu at (233.2, 65.2)
- added R70: 39k, easyeda2kicad:R0402, B.Cu at (230.3, 54.0)
- added R71: 10k, easyeda2kicad:R0402, B.Cu at (227.4, 59.9)
- added R72: 10k, easyeda2kicad:R0402, B.Cu at (228.9, 44.7)
- added R73: 10k, easyeda2kicad:R0402, B.Cu at (226.6, 44.3)
- added R74: 50k, easyeda2kicad:R0402, B.Cu at (227.6, 44.3)
- added U3: STDRIVE101, easyeda2kicad:QFN-24_L4.0-W4.0-P0.50-BL-EP2.7, F.Cu at (232.0, 51.5)
- added U4: STDRIVE101, easyeda2kicad:QFN-24_L4.0-W4.0-P0.50-BL-EP2.7, F.Cu at (230.0, 69.0)
- added U5: STM32C011F6U6TR, easyeda2kicad:UFQFPN-20_L3.0-W3.0-P0.50-TL, F.Cu at (230.0, 74.3)
- added U6: STDRIVE101, easyeda2kicad:QFN-24_L4.0-W4.0-P0.50-BL-EP2.7, B.Cu at (230.0, 69.0)
- added U7: STM32C011F6U6TR, easyeda2kicad:UFQFPN-20_L3.0-W3.0-P0.50-TL, B.Cu at (230.0, 74.3)
- added U8: STDRIVE101, easyeda2kicad:QFN-24_L4.0-W4.0-P0.50-BL-EP2.7, B.Cu at (228.0, 51.5)
- added U9: STM32C011F6U6TR, easyeda2kicad:UFQFPN-20_L3.0-W3.0-P0.50-TL, B.Cu at (228.2, 56.8)
- C10: value 100nF -> 1uF
- C11: value 4.7uF -> 100nF
- C15: value 100nF -> 4.7uF; footprint easyeda2kicad:C0402 -> easyeda2kicad:C0603; moved to F.Cu
- C16: value 1uF -> 100nF; footprint easyeda2kicad:C0603 -> easyeda2kicad:C0402; moved to F.Cu
- C17: value 0.1uF -> 4.7uF; footprint easyeda2kicad:C0603 -> easyeda2kicad:C0402; moved to F.Cu
- C18: value 100nF -> 1uF; moved to F.Cu
- C19: value >10uF -> 1uF; footprint easyeda2kicad:C0603 -> easyeda2kicad:C0402; moved to F.Cu
- C20: value 0.1uF -> 100nF; moved to F.Cu
- C21: footprint easyeda2kicad:C0603 -> easyeda2kicad:C0402; moved to F.Cu
- C22: value 47nF -> 100nF; moved to B.Cu
- C23, C39: value 1uF -> 100nF; footprint easyeda2kicad:C0603 -> easyeda2kicad:C0402; moved to B.Cu
- C24, C25, C26, C48, C49, C50, Q11, Q13, Q15, Q17, Q7, Q9, R15, R16, R17, R18, R19, R20, R56, R57, R58, R59, R60, R61, R7: moved to F.Cu
- C27: value >10uF -> 100nF; footprint easyeda2kicad:C0603 -> easyeda2kicad:C0402
- C28: value 0.1uF -> 4.7uF; footprint easyeda2kicad:C0402 -> easyeda2kicad:C0603
- C29, C37: value 1uF -> 100nF; footprint easyeda2kicad:C0603 -> easyeda2kicad:C0402
- C30: value 47nF -> 4.7uF; footprint easyeda2kicad:C0603 -> easyeda2kicad:C0402; moved to B.Cu
- C31: footprint easyeda2kicad:C0603 -> easyeda2kicad:C0402; moved to B.Cu
- C35: value >10uF -> 100nF
- C36: value 0.1uF -> 100nF
- C38: value 47nF -> 4.7uF
- C43: value >10uF -> 1uF; footprint easyeda2kicad:C0603 -> easyeda2kicad:C0402
- C44: value 0.1uF -> 1uF
- C45: value 1uF -> 4.7uF; footprint easyeda2kicad:C0603 -> easyeda2kicad:C0402
- C46: value 47nF -> 1uF; footprint easyeda2kicad:C0603 -> easyeda2kicad:C0402; moved to B.Cu
- C47: footprint easyeda2kicad:C0603 -> easyeda2kicad:C0402
- C51, C52, C54, Q10, Q12, Q14, Q16, Q18, Q8, R24, R26, R28, R38, R40, R42: moved to B.Cu
- C6: value 5pF-25pF -> 100nF; footprint easyeda2kicad:C0402 -> easyeda2kicad:C0603; moved to F.Cu
- C7: value 5pF-25pF -> 4.7uF; footprint easyeda2kicad:C0402 -> easyeda2kicad:C0603; moved to F.Cu
- C8, C9: value 2.2uF -> 1uF
- R21: value 10k -> 18k
- R22: value 10k -> 39k; moved to B.Cu
- R3: value 10k -> 50k
- R36: value 10k -> 18k; moved to B.Cu
- R4: value 10K -> 18k; moved to F.Cu
- R49, R8: value 10k -> 39k
- R5: value 5K1 -> 18k; moved to F.Cu
- R6: value 5K1 -> 10k; moved to F.Cu
- U2: value STM32F405RGT6 -> STM32C011F6U6TR; footprint easyeda2kicad:LQFP-64_L10.0-W10.0-P0.50-LS12.0-BL -> easyeda2kicad:UFQFPN-20_L3.0-W3.0-P0.50-TL
- moved C50 29.5 mm to (261.7, 65.2), turned to -90 degrees
- moved C46 28.8 mm to (225.7, 47.8), turned to 0 degrees
- moved R61 28.4 mm to (260.8, 65.1), turned to 90 degrees
- moved R30 28.1 mm to (196.8, 69.4), turned to 90 degrees
- moved R43 27.7 mm to (197.1, 52.3), turned to 90 degrees
- moved R29 26.8 mm to (196.8, 67.5), turned to 90 degrees
- moved R44 26.6 mm to (197.1, 54.2), turned to 90 degrees
- moved R60 26.4 mm to (260.8, 63.2), turned to 90 degrees
- moved C23 26.0 mm to (234.5, 68.8)
- moved C32 26.0 mm to (198.0, 69.4), turned to -90 degrees
- moved R5 25.9 mm to (226.6, 62.8), turned to 180 degrees
- moved C40 25.4 mm to (198.0, 54.2), turned to -90 degrees
- moved C26 25.0 mm to (259.0, 47.4), turned to -90 degrees
- moved R20 24.0 mm to (257.9, 47.4), turned to 90 degrees
- moved C48 23.4 mm to (254.2, 64.9)
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Connections:
- net GHA1 renamed Net-(Q1-G)
- net GHA2 renamed Net-(Q7-G)
- net GHA3 renamed Net-(Q13-G)
- net GHA4 renamed Net-(Q19-G)
- net GHB1 renamed Net-(Q3-G)
- net GHB2 renamed Net-(Q9-G)
- net GHB3 renamed Net-(Q15-G)
- net GHB4 renamed Net-(Q21-G)
- net GHC1 renamed Net-(Q5-G)
- net GHC2 renamed Net-(Q11-G)
- net GHC3 renamed Net-(Q17-G)
- net GHC4 renamed Net-(Q23-G)
- net GLA1 renamed Net-(Q2-G)
- net GLA2 renamed Net-(Q8-G)
- net GLA3 renamed Net-(Q14-G)
- net GLA4 renamed Net-(Q20-G)
- net GLB1 renamed Net-(Q4-G)
- net GLB2 renamed Net-(Q10-G)
- net GLB3 renamed Net-(Q16-G)
- net GLB4 renamed Net-(Q22-G)
- net GLC1 renamed Net-(Q6-G)
- net GLC2 renamed Net-(Q12-G)
- net GLC3 renamed Net-(Q18-G)
- net GLC4 renamed Net-(Q24-G)
- C10 pad 1: GND -> OUT3
- C10 pad 2: 3V3 -> Net-(U3-BOOT3)
- C11 pad 1: GND -> Net-(U4-REG12)
- C11 pad 2: 3V3 -> GND
- C12 pad 1: GND -> 3V3
- C12 pad 2: 3V3 -> GND
- C13 pad 1: GND -> B+
- C13 pad 2: 3V3 -> GND
- C14 pad 1: GND -> 3V3
- C14 pad 2: 3V3 -> GND
- C15 pad 1: 3V3 -> Net-(U4-REG12)
- C16 pad 1: 3V3 -> Net-(U5-PF2-NRST)
- C17 pad 1: RESET -> 3V3
- C18 pad 1: BOOT0 -> OUT1
- C18 pad 2: GND -> Net-(U4-BOOT1)
- C19 pad 1: B+ -> OUT2
- C19 pad 2: GND -> Net-(U4-BOOT2)
- C21 pad 1: B+ -> OUT3
- C22 pad 1: Net-(M1-CPL) -> Net-(U6-REG12)
- C22 pad 2: Net-(M1-CPH) -> GND
- C23 pad 1: Net-(M1-DVDD) -> B+
- C27 pad 1: B+ -> 3V3
- C28 pad 1: B+ -> Net-(U6-REG12)
- C29 pad 1: B+ -> Net-(U7-PF2-NRST)
- C29 pad 2: Net-(M2-VCP) -> GND
- C30 pad 1: Net-(M2-CPL) -> 3V3
- C30 pad 2: Net-(M2-CPH) -> GND
- C31 pad 1: Net-(M2-DVDD) -> OUT1
- C31 pad 2: GND -> Net-(U6-BOOT1)
- C35 pad 1: B+ -> Net-(U8-REG12)
- C37 pad 1: B+ -> 3V3
- C37 pad 2: Net-(M3-VCP) -> GND
- C38 pad 1: Net-(M3-CPL) -> Net-(U8-REG12)
- C38 pad 2: Net-(M3-CPH) -> GND
- C43 pad 1: B+ -> OUT2
- C43 pad 2: GND -> Net-(U6-BOOT2)
- C44 pad 1: B+ -> OUT3
- C44 pad 2: GND -> Net-(U6-BOOT3)
- C45 pad 1: B+ -> 3V3
- C45 pad 2: Net-(M4-VCP) -> GND
- C46 pad 1: Net-(M4-CPL) -> OUT1
- C47 pad 1: Net-(M4-DVDD) -> OUT2
- C47 pad 2: GND -> Net-(U8-BOOT2)
- C6 pad 1: Net-(U2A-PH0-OSC_IN(PH0)) -> Net-(U3-REG12)
- C7 pad 1: GND -> Net-(U3-REG12)
- C7 pad 2: Net-(U2A-PH1-OSC_OUT(PH1)) -> GND
- C8 pad 1: GND -> OUT1
- C8 pad 2: Net-(U2A-VCAP_1) -> Net-(U3-BOOT1)
- C9 pad 1: GND -> OUT2
- C9 pad 2: Net-(U2A-VCAP_2) -> Net-(U3-BOOT2)
- J10 pad 1: SHA3 -> OUT1
- J11 pad 1: SHB3 -> OUT2
- J12 pad 1: SHC3 -> OUT3
- J13 pad 1: SHA4 -> OUT1
- J14 pad 1: SHB4 -> OUT2
- J15 pad 1: SHC4 -> OUT3
- J2 pad 1: DShot -> DShot_M1
- J4 pad 1: SHA1 -> OUT1
- J5 pad 1: SHB1 -> OUT2
- J6 pad 1: SHC1 -> OUT3
- J7 pad 1: SHA2 -> OUT1
- J8 pad 1: SHB2 -> OUT2
- J9 pad 1: SHC2 -> OUT3
- Q1 pad 1: SHA1 -> OUT1
- Q1 pad 2: SHA1 -> OUT1
- Q1 pad 3: SHA1 -> OUT1
- Q10 pad 5: SHB2 -> OUT2
- Q10 pad 6: SHB2 -> OUT2
- Q10 pad 7: SHB2 -> OUT2
- Q10 pad 8: SHB2 -> OUT2
- Q10 pad 9: SHB2 -> OUT2
- Q11 pad 1: SHC2 -> OUT3
- Q11 pad 2: SHC2 -> OUT3
- Q11 pad 3: SHC2 -> OUT3
- Q12 pad 5: SHC2 -> OUT3
- Q12 pad 6: SHC2 -> OUT3
- Q12 pad 7: SHC2 -> OUT3
- Q12 pad 8: SHC2 -> OUT3
- Q12 pad 9: SHC2 -> OUT3
- Q13 pad 1: SHA3 -> OUT1
- Q13 pad 2: SHA3 -> OUT1
- Q13 pad 3: SHA3 -> OUT1
- Q14 pad 5: SHA3 -> OUT1
- Q14 pad 6: SHA3 -> OUT1
- Q14 pad 7: SHA3 -> OUT1
- Q14 pad 8: SHA3 -> OUT1
- Q14 pad 9: SHA3 -> OUT1
- Q15 pad 1: SHB3 -> OUT2
- Q15 pad 2: SHB3 -> OUT2
- Q15 pad 3: SHB3 -> OUT2
- Q16 pad 5: SHB3 -> OUT2
- Q16 pad 6: SHB3 -> OUT2
- Q16 pad 7: SHB3 -> OUT2
- Q16 pad 8: SHB3 -> OUT2
- Q16 pad 9: SHB3 -> OUT2
- Q17 pad 1: SHC3 -> OUT3
- Q17 pad 2: SHC3 -> OUT3
- Q17 pad 3: SHC3 -> OUT3
- Q18 pad 5: SHC3 -> OUT3
- Q18 pad 6: SHC3 -> OUT3
- Q18 pad 7: SHC3 -> OUT3
- Q18 pad 8: SHC3 -> OUT3
- Q18 pad 9: SHC3 -> OUT3
- Q19 pad 1: SHA4 -> OUT1
- Q19 pad 2: SHA4 -> OUT1
- Q19 pad 3: SHA4 -> OUT1
- Q2 pad 5: SHA1 -> OUT1
- Q2 pad 6: SHA1 -> OUT1
- Q2 pad 7: SHA1 -> OUT1
- Q2 pad 8: SHA1 -> OUT1
- Q2 pad 9: SHA1 -> OUT1
- Q20 pad 5: SHA4 -> OUT1
- Q20 pad 6: SHA4 -> OUT1
- Q20 pad 7: SHA4 -> OUT1
- Q20 pad 8: SHA4 -> OUT1
- Q20 pad 9: SHA4 -> OUT1
- Q21 pad 1: SHB4 -> OUT2
- Q21 pad 2: SHB4 -> OUT2
- Q21 pad 3: SHB4 -> OUT2
- Q22 pad 5: SHB4 -> OUT2
- Q22 pad 6: SHB4 -> OUT2
- Q22 pad 7: SHB4 -> OUT2
- Q22 pad 8: SHB4 -> OUT2
- Q22 pad 9: SHB4 -> OUT2
- Q23 pad 1: SHC4 -> OUT3
- Q23 pad 2: SHC4 -> OUT3
- Q23 pad 3: SHC4 -> OUT3
- Q24 pad 5: SHC4 -> OUT3
- Q24 pad 6: SHC4 -> OUT3
- Q24 pad 7: SHC4 -> OUT3
- Q24 pad 8: SHC4 -> OUT3
- Q24 pad 9: SHC4 -> OUT3
- Q3 pad 1: SHB1 -> OUT2
- Q3 pad 2: SHB1 -> OUT2
- Q3 pad 3: SHB1 -> OUT2
- Q4 pad 5: SHB1 -> OUT2
- Q4 pad 6: SHB1 -> OUT2
- Q4 pad 7: SHB1 -> OUT2
- Q4 pad 8: SHB1 -> OUT2
- Q4 pad 9: SHB1 -> OUT2
- Q5 pad 1: SHC1 -> OUT3
- Q5 pad 2: SHC1 -> OUT3
- Q5 pad 3: SHC1 -> OUT3
- Q6 pad 5: SHC1 -> OUT3
- Q6 pad 6: SHC1 -> OUT3
- Q6 pad 7: SHC1 -> OUT3
- Q6 pad 8: SHC1 -> OUT3
- Q6 pad 9: SHC1 -> OUT3
- Q7 pad 1: SHA2 -> OUT1
- Q7 pad 2: SHA2 -> OUT1
- Q7 pad 3: SHA2 -> OUT1
- Q8 pad 5: SHA2 -> OUT1
- Q8 pad 6: SHA2 -> OUT1
- Q8 pad 7: SHA2 -> OUT1
- Q8 pad 8: SHA2 -> OUT1
- Q8 pad 9: SHA2 -> OUT1
- Q9 pad 1: SHB2 -> OUT2
- Q9 pad 2: SHB2 -> OUT2
- Q9 pad 3: SHB2 -> OUT2
- R10 pad 2: GND -> GLS1
- R11 pad 2: SHB1 -> GHS2
- R12 pad 2: GND -> GLS2
- R13 pad 2: SHC1 -> GHS3
- R14 pad 2: GND -> GLS3
- R15 pad 2: SHA1 -> OUT1
- R17 pad 2: SHB1 -> OUT2
- R19 pad 2: SHC1 -> OUT3
- R21 pad 2: PUPL2 -> Net-(U6-SCREF)
- R23 pad 2: SHA2 -> GHS1
- R24 pad 2: GND -> GLS1
- R25 pad 2: SHB2 -> GHS2
- R26 pad 2: GND -> GLS2
- R27 pad 2: SHC2 -> GHS3
- R28 pad 2: GND -> GLS3
- R29 pad 2: SHA2 -> OUT1
- R3 pad 1: SDO -> Net-(U3-DT/MODE)
- R3 pad 2: 3V3 -> GND
- R31 pad 2: SHB2 -> OUT2
- R33 pad 2: SHC2 -> OUT3
- R36 pad 1: Net-(M3-nFAULT) -> 3V3
- R36 pad 2: 3V3 -> Net-(U8-SCREF)
- R37 pad 2: SHA3 -> GHS1
- R38 pad 2: GND -> GLS1
- R39 pad 2: SHB3 -> GHS2
- R4 pad 1: BOOT0 -> 3V3
- R4 pad 2: GND -> Net-(U3-SCREF)
- R40 pad 2: GND -> GLS2
- R41 pad 2: SHC3 -> GHS3
- R42 pad 2: GND -> GLS3
- R43 pad 2: SHA3 -> OUT1
- R45 pad 2: SHB3 -> OUT2
- R47 pad 2: SHC3 -> OUT3
- R5 pad 1: GND -> 3V3
- R50 pad 2: SHA4 -> GHS1
- R51 pad 2: GND -> GLS1
- R52 pad 2: SHB4 -> GHS2
- R53 pad 2: GND -> GLS2
- R54 pad 2: SHC4 -> GHS3
- R55 pad 2: GND -> GLS3
- R56 pad 2: SHA4 -> OUT1
- R58 pad 2: SHB4 -> OUT2
- R6 pad 1: GND -> Net-(U2-PF2-NRST)
- R6 pad 2: Net-(USBC1-CC2) -> 3V3
- R60 pad 2: SHC4 -> OUT3
- R7 pad 1: 3V3 -> Net-(U3-SCREF)
- R7 pad 2: PUPL1 -> GND
- R9 pad 2: SHA1 -> GHS1
- U2 pad 1: 3V3 -> unconnected-(U2-PC15-OSCX_OUT-Pad1)
- U2 pad 10: INHC_M2 -> EN3_M1
- U2 pad 11: EN_M4 -> EN2_M1
- U2 pad 12: GND -> EN1_M1
- U2 pad 13: 3V3 -> INH3_M1
- U2 pad 14: INHC_M4 -> INH2_M1
- U2 pad 15: INHB_M4 -> INH1_M1
- U2 pad 16: INHA_M4 -> SWDIO_M1
- U2 pad 17: CS_M4 -> SWCLK
- U2 pad 18: GND -> unconnected-(U2-PB6-Pad18)
- U2 pad 19: 3V3 -> unconnected-(U2-PB7-Pad19)
- U2 pad 2: CS_M2 -> 3V3
- U2 pad 20: PHASE_A_M4 -> unconnected-(U2-PC14-OSCX_IN-Pad20)
- U2 pad 3: EN_M2 -> GND
- U2 pad 4: unconnected-(U2A-PC15-OSC32_OUT(PC15)-Pad4) -> Net-(U2-PF2-NRST)
- U2 pad 5: Net-(U2A-PH0-OSC_IN(PH0)) -> unconnected-(U2-PA0-Pad5)
- U2 pad 6: Net-(U2A-PH1-OSC_OUT(PH1)) -> unconnected-(U2-PA1-Pad6)
- U2 pad 7: RESET -> PHASE_B_M1
- U2 pad 8: INHB_M2 -> PHASE_A_M1
- U2 pad 9: INHA_M2 -> PHASE_C_M1
Routing:
- net GND: track 188.4 -> 7.89 mm, vias 113 -> 112
- net GHS1: track 0.00 -> 55.6 mm, vias 0 -> 1
- net GHS3: track 0.00 -> 51.1 mm, vias 0 -> 1
- net GHS2: track 0.00 -> 49.1 mm, vias 0 -> 1
- net SHC4: track 34.9 -> 0.00 mm, vias 11 -> 0
- net BOOT0: track 34.6 -> 0.00 mm, vias 2 -> 0
- net GLS1: track 0.00 -> 33.0 mm, vias 0 -> 2
- net RESET: track 26.1 -> 0.00 mm, vias 3 -> 0
- net Net-(Q23-G): track 24.8 -> 0.00 mm, vias 3 -> 0
- net GLS2: track 0.00 -> 24.6 mm, vias 0 -> 2
- net GLS3: track 0.00 -> 24.5 mm, vias 0 -> 2
- net OUT1: track 0.00 -> 23.1 mm, vias 0 -> 17
- net DShot: track 21.8 -> 0.00 mm, vias 2 -> 0
- net SHC3: track 21.5 -> 0.00 mm, vias 10 -> 0
- net PHASE_A_M3: track 21.4 -> 0.00 mm, vias 1 -> 0
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- removed copper zone on In3.Cu, net 3V3
- removed copper zone on B.Cu, net SHA1
- removed copper zone on F.Cu, net SHA1
- removed copper zone on B.Cu, net SHA2
- removed copper zone on F.Cu, net SHA2
- removed copper zone on B.Cu, net SHA3
- removed copper zone on F.Cu, net SHA3
- removed copper zone on B.Cu, net SHA4
- removed copper zone on F.Cu, net SHA4
- removed copper zone on B.Cu, net SHB1
- removed copper zone on F.Cu, net SHB1
- removed copper zone on B.Cu, net SHB2
- removed copper zone on F.Cu, net SHB2
- removed copper zone on B.Cu, net SHB3
- removed copper zone on F.Cu, net SHB3
- removed copper zone on B.Cu, net SHB4
- removed copper zone on F.Cu, net SHB4
- removed copper zone on B.Cu, net SHC1
- removed copper zone on F.Cu, net SHC1
- removed copper zone on B.Cu, net SHC2
- removed copper zone on F.Cu, net SHC2
- removed copper zone on B.Cu, net SHC3
- removed copper zone on F.Cu, net SHC3
- removed copper zone on B.Cu, net SHC4
- removed copper zone on F.Cu, net SHC4
Other:
- board size 40 x 50 mm -> 40 x 45 mm
- copper layers 6 -> 4

Commit message: ...
Parts:
- C10, C12, C20, C55, C56, C6, C7, C8, C9, J18, J2, R3, R35, R4, R6, R7, R8, U2, U3: moved to B.Cu
- C35, C36, C37, C38, C39, C45, C46, C47, C51, C52, C54, C57, C58, C59, C62, C63, C64, C65, R36, R70, R71, R72, R73, R74, U8, U9: moved to F.Cu
- moved C40 29.3 mm to (225.2, 43.2), turned to 90 degrees
- moved R44 29.3 mm to (224.3, 43.2), turned to -90 degrees
- moved R43 27.8 mm to (223.3, 43.2)
- moved R46 27.1 mm to (226.7, 45.3), turned to 180 degrees
- moved R45 26.8 mm to (226.7, 44.3), turned to 0 degrees
- moved C41 26.0 mm to (226.7, 46.2), turned to 0 degrees
- moved R47 20.9 mm to (225.2, 47.1), turned to -90 degrees
- moved R48 20.5 mm to (224.3, 47.1)
- moved C42 18.7 mm to (223.4, 47.1)
- moved C55 17.9 mm to (231.2, 42.5)
- moved C45 17.9 mm to (228.9, 42.5)
- moved C39 17.0 mm to (227.5, 43.0), turned to 90 degrees
- moved R71 17.0 mm to (226.6, 43.0), turned to 90 degrees
- moved C56 17.0 mm to (232.5, 43.0), turned to 90 degrees
- moved R6 17.0 mm to (233.4, 43.0), turned to 90 degrees
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Connections:
- U2 pad 17: SWCLK -> SWCLK_H
- U2 pad 6: unconnected-(U2-PA1-Pad6) -> DShot_M1
- U2 pad 7: PHASE_B_M1 -> PHASE_A_M1
- U2 pad 8: PHASE_A_M1 -> PHASE_B_M1
- U5 pad 17: SWCLK -> SWCLK_L
- U5 pad 6: unconnected-(U5-PA1-Pad6) -> DShot_M4
- U5 pad 7: unconnected-(U5-PA2-Pad7) -> PHASE_B_M1
- U5 pad 8: unconnected-(U5-PA3-Pad8) -> PHASE_A_M1
- U5 pad 9: unconnected-(U5-PA4-Pad9) -> PHASE_C_M1
- U7 pad 17: SWCLK -> SWCLK_L
- U7 pad 6: unconnected-(U7-PA1-Pad6) -> DShot_M2
- U7 pad 7: unconnected-(U7-PA2-Pad7) -> PHASE_B_M1
- U7 pad 8: unconnected-(U7-PA3-Pad8) -> PHASE_A_M1
- U7 pad 9: unconnected-(U7-PA4-Pad9) -> PHASE_C_M1
- U9 pad 17: SWCLK -> SWCLK_H
- U9 pad 6: unconnected-(U9-PA1-Pad6) -> DShot_M3
- U9 pad 7: unconnected-(U9-PA2-Pad7) -> PHASE_B_M1
- U9 pad 8: unconnected-(U9-PA3-Pad8) -> PHASE_A_M1
- U9 pad 9: unconnected-(U9-PA4-Pad9) -> PHASE_C_M1
Routing:
- net OUT1: track 23.1 -> 91.4 mm, vias 17 -> 44
- net OUT2: track 7.14 -> 75.0 mm, vias 9 -> 44
- net OUT3: track 13.4 -> 76.0 mm, vias 9 -> 44
- net GHS1: track 55.6 -> 73.9 mm, vias 1 -> 2
- net B+: track 17.9 -> 33.4 mm
- net GHS2: track 49.1 -> 63.4 mm, vias 1 -> 2
- net GHS3: track 51.1 -> 61.2 mm, vias 1 -> 2
- net GLS1: track 33.0 -> 42.8 mm, vias 2 -> 4
- net GLS3: track 24.5 -> 33.3 mm, vias 2 -> 4
- net Net-(U6-REG12): track 0.00 -> 8.76 mm
- net GLS2: track 24.6 -> 33.2 mm, vias 2 -> 4
- net DShot_M3: track 0.00 -> 6.52 mm
- net DShot_M1: track 0.00 -> 6.49 mm
- net DShot_M4: track 0.00 -> 6.28 mm
- net DShot_M2: track 0.00 -> 6.28 mm
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- added copper zone on In4.Cu, net 3V3
Other:
- copper layers 4 -> 6
