File: esc.kicad_pcb (KiCad board)
At the start: 6 copper layers, 40 x 45 mm, 188 parts, among them J1 Conn_01x02, J10 Conn_01x01_Pin, J11 Conn_01x01_Pin, J12 Conn_01x01_Pin, J13 Conn_01x01_Pin, J14 Conn_01x01_Pin, J15 Conn_01x01_Pin, J16 Conn_01x02, J17 Conn_01x01_Pin, J18 Conn_01x01_Pin, J19 Conn_01x01_Pin, J2 Conn_01x01_Pin, J20 Conn_01x01_Pin, J4 Conn_01x01_Pin, J5 Conn_01x01_Pin, J6 Conn_01x01_Pin, J7 Conn_01x01_Pin, J8 Conn_01x01_Pin, J9 Conn_01x01_Pin, Q1 NP80N06D6, Q10 NP80N06D6, Q11 NP80N06D6, Q12 NP80N06D6, Q13 NP80N06D6, Q14 NP80N06D6, Q15 NP80N06D6, Q16 NP80N06D6, Q17 NP80N06D6, Q18 NP80N06D6, Q19 NP80N06D6, Q2 NP80N06D6, Q20 NP80N06D6, Q21 NP80N06D6, Q22 NP80N06D6, Q23 NP80N06D6, Q24 NP80N06D6, Q3 NP80N06D6, Q4 NP80N06D6, Q5 NP80N06D6, Q6 NP80N06D6, Q7 NP80N06D6, Q8 NP80N06D6, Q9 NP80N06D6, U2 STM32C011F6U6TR, U3 STDRIVE101, U4 STDRIVE101, U5 STM32C011F6U6TR, U6 STDRIVE101, U7 STM32C011F6U6TR, U8 STDRIVE101, U9 STM32C011F6U6TR

Commit message: ...
Parts:
- added J21: Conn_01x01_Pin, deshan:Conn_01x01_Pin, B.Cu at (222.0, 40.9)
- added J22: Conn_01x01_Pin, deshan:Conn_01x01_Pin, B.Cu at (240.0, 79.2)
- added J23: Conn_01x01_Pin, deshan:Conn_01x01_Pin, B.Cu at (238.0, 79.2)
- added J24: ~, deshan:Conn_01x01_Pin, F.Cu at (240.0, 40.9)
- added J25: Conn_01x01_Pin, deshan:Conn_01x01_Pin, F.Cu at (220.0, 79.2)
- added J26: Conn_01x01_Pin, deshan:Conn_01x01_Pin, F.Cu at (238.0, 40.9)
- added J27: Conn_01x01_Pin, deshan:Conn_01x01_Pin, F.Cu at (222.0, 79.2)
- added J3: Conn_01x01_Pin, deshan:Conn_01x01_Pin, B.Cu at (220.0, 40.9)
- C28: renamed from C32; moved to F.Cu
- C29: renamed from C33; moved to F.Cu
- C30: renamed from C34; moved to F.Cu
- C58: renamed from C48; moved to B.Cu
- C59: renamed from C49; moved to B.Cu
- C60: renamed from C50; moved to B.Cu
- J10, J11, J12, J13, J14, J15, J4, J5, J6, J7, J8, J9: footprint deshan:Conn_1x1 -> deshan:Conn_01x01_Power
- J18, J19, J2, J20: footprint deshan:Conn_1x1_small -> deshan:Conn_01x01_Pin
- R31: renamed from R29; moved to F.Cu
- R32: renamed from R30; moved to F.Cu
- R33: renamed from R31; moved to F.Cu
- R34: renamed from R32; moved to F.Cu
- R35: renamed from R33; moved to F.Cu
- R36: renamed from R34; moved to F.Cu
- R67: renamed from R56; moved to B.Cu
- R68: renamed from R57; moved to B.Cu
- R69: renamed from R58; moved to B.Cu
- R70: renamed from R59; moved to B.Cu
- R71: renamed from R60; moved to B.Cu
- R72: renamed from R61; moved to B.Cu
- moved C28 29.9 mm to (225.6, 72.8), turned to 90 degrees
- moved R71 29.1 mm to (234.5, 75.7), turned to -90 degrees
- moved R32 28.0 mm to (224.6, 72.8), turned to -90 degrees
- moved C29 28.0 mm to (227.7, 75.2), turned to 0 degrees
- moved R72 27.5 mm to (235.4, 75.7)
- moved C60 27.4 mm to (236.4, 75.7)
- moved C59 27.1 mm to (232.6, 75.1), turned to 180 degrees
- moved R34 26.9 mm to (227.7, 74.3), turned to 180 degrees
- moved R69 26.3 mm to (232.6, 73.2), turned to 180 degrees
- moved R31 26.2 mm to (223.7, 72.8), turned to 90 degrees
- moved R70 25.9 mm to (232.6, 74.2), turned to 0 degrees
- moved R33 25.8 mm to (227.7, 73.3), turned to 0 degrees
- moved C15 24.6 mm to (234.7, 43.5), turned to 90 degrees
- moved C14 23.6 mm to (233.0, 44.9), turned to 180 degrees
- moved R18 22.6 mm to (235.6, 43.5), turned to -90 degrees
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- renumbered C56 to C1, C51 to C10, C58 to C11, C59 to C12, C24 to C13, C25 to C14, C26 to C15, C29 to C16, C27 to C17, C30 to C18, C23 to C19, C12 to C2, C22 to C20, C28 to C21, C31 to C22, C43 to C23, C44 to C24, C52 to C25, C64 to C26, C65 to C27, C55 to C3, C39 to C31, C37 to C32, C45 to C33, C36 to C34, C38 to C36, C46 to C37, C47 to C38, C57 to C39, C20 to C4, C53 to C40, C61 to C41, C60 to C42, C40 to C43, C41 to C44, C42 to C45, C16 to C46, C14 to C47, C17 to C48, C13 to C49, C6 to C5, C11 to C50, C15 to C51, C18 to C52, C19 to C53, C21 to C54, C54 to C55, C62 to C56, C63 to C57, C7 to C6, C8 to C7, C9 to C8, C10 to C9, R6 to R1, R12 to R10, R13 to R11, R14 to R12, R15 to R13, R16 to R14, R17 to R15, R18 to R16, R19 to R17, R20 to R18, R66 to R19, R4 to R2, R21 to R20, R67 to R21, R68 to R22, R69 to R23, R22 to R24, R23 to R25, R24 to R26, R25 to R27, R26 to R28, R27 to R29, R7 to R3, R28 to R30, R71 to R37, R36 to R38, R72 to R39, R35 to R4, R73 to R40, R74 to R41, R70 to R42, R37 to R43, R38 to R44, R39 to R45, R40 to R46, R41 to R47, R42 to R48, R43 to R49, R3 to R5, R44 to R50, R45 to R51, R46 to R52, R47 to R53, R48 to R54, R62 to R55, R5 to R56, R63 to R57, R64 to R58, R65 to R59, R8 to R6, R49 to R60, R50 to R61, R51 to R62, R52 to R63, R53 to R64, R54 to R65, R55 to R66, R9 to R7, R10 to R8, R11 to R9
Connections:
- U2 pad 17: SWCLK_H -> SWCLK_M1
- U2 pad 7: PHASE_A_M1 -> PHASE_C_M1
- U2 pad 9: PHASE_C_M1 -> PHASE_A_M1
- U5 pad 17: SWCLK_L -> SWCLK_M4
- U5 pad 7: PHASE_B_M1 -> PHASE_C_M4
- U5 pad 8: PHASE_A_M1 -> PHASE_B_M4
- U5 pad 9: PHASE_C_M1 -> PHASE_A_M4
- U7 pad 17: SWCLK_L -> SWCLK_M2
- U7 pad 7: PHASE_B_M1 -> PHASE_C_M2
- U7 pad 8: PHASE_A_M1 -> PHASE_B_M2
- U7 pad 9: PHASE_C_M1 -> PHASE_A_M2
- U9 pad 17: SWCLK_H -> SWCLK_M3
- U9 pad 7: PHASE_B_M1 -> PHASE_C_M3
- U9 pad 8: PHASE_A_M1 -> PHASE_B_M3
- U9 pad 9: PHASE_C_M1 -> PHASE_A_M3
Routing:
- net OUT1: track 91.4 -> 155.6 mm
- net OUT3: track 76.0 -> 119.6 mm
- net OUT2: track 75.0 -> 99.3 mm
- net SWDIO_M3: track 0.00 -> 16.6 mm
- net SWDIO_M1: track 0.00 -> 16.4 mm
- net SWDIO_M2: track 0.00 -> 14.6 mm
- net SWDIO_M4: track 0.00 -> 14.0 mm
- net GND: track 12.5 -> 26.3 mm, vias 108 -> 124
- net SWCLK_M3: track 0.00 -> 13.6 mm
- net SWCLK_M1: track 0.00 -> 13.5 mm
- net SWCLK_M2: track 0.00 -> 12.4 mm
- net SWCLK_M4: track 0.00 -> 11.8 mm
- net PHASE_B_M1: track 0.00 -> 6.29 mm, vias 0 -> 1
- net PHASE_B_M2: track 0.00 -> 6.10 mm, vias 0 -> 1
- net PHASE_B_M3: track 0.00 -> 5.70 mm, vias 0 -> 1
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