File: esc.kicad_sch (KiCad schematic)
At the start: 0 parts

Commit message: ...
Other:
- sheet MCU renamed GPIO-CONN
- sheet GPIO-CONN: file mcu.kicad_sch -> gpio-conn.kicad_sch
- title: (none) -> ESC MULTI-MCU-ARCHITECTURE
Changed lines of the file:
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@@
 	(generator_version "10.0")
 	(paper "A4")
+	(title_block
+		(title "ESC MULTI-MCU-ARCHITECTURE")
+		(rev "1.0")
+		(comment 1 "This is the pcb for an Elettronic Speed Controller of 4 indipendent BLDC motors.")
+		(comment 2 "MAX SPECIFICATION: 30V - 50A, Logic Level 3v3.")
+	)
 	(sheet
 		(at 152.4 58.42)
@@
 			(color 0 0 0 0)
 		)
-		(property "Sheetname" "MCU"
+		(property "Sheetname" "GPIO-CONN"
 			(at 91.44 108.5084 0)
 			(show_name no)
@@
 			)
 		)
-		(property "Sheetfile" "mcu.kicad_sch"
+		(property "Sheetfile" "gpio-conn.kicad_sch"
 			(at 91.44 135.2046 0)
 			(show_name no)

Commit message: ...
Other:
- removed sheet GPIO-CONN
- note added: "ELECTRONIC SPEED CONTROLLER 4in1"
- note added: "MAX SPECIFICATION : 60V - 12A (PEAK) LOGIC LEVEL : 3V3"
Changed lines of the file:
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@@
 		(title "ESC MULTI-MCU-ARCHITECTURE")
 		(rev "1.0")
-		(comment 1 "This is the pcb for an Elettronic Speed Controller of 4 indipendent BLDC motors.")
-		(comment 2 "MAX SPECIFICATION: 30V - 50A, Logic Level 3v3.")
-	)
-	(sheet
-		(at 152.4 58.42)
+	)
+	(text "MAX SPECIFICATION : 60V - 12A (PEAK) \nLOGIC LEVEL : 3V3 "
+		(exclude_from_sim no)
+		(at 177.546 173.482 0)
+		(effects
+			(font
+				(size 1.27 1.27)
+				(thickness 0.254)
+				(bold yes)
+			)
+			(justify left)
+		)
+	)
+	(text "ELECTRONIC SPEED CONTROLLER 4in1"
+		(exclude_from_sim no)
+		(at 195.834 168.656 0)
+		(effects
+			(font
+				(size 1.27 1.27)
+				(thickness 0.254)
+				(bold yes)
+			)
+		)
+	)
+	(sheet
+		(at 35.56 91.44)
 		(size 31.75 26.67)
 		(exclude_from_sim no)
@@
 		)
 		(property "Sheetname" "MOTOR_DRIVER_M3"
-			(at 152.4 57.7084 0)
+			(at 35.56 90.7284 0)
 			(show_name no)
 			(do_not_autoplace no)
@@
 		)
 		(property "Sheetfile" "motor_driver_m3.kicad_sch"
-			(at 152.4 85.6746 0)
+			(at 35.56 118.6946 0)
 			(show_name no)
 			(do_not_autoplace no)
@@
 	)
 	(sheet
-		(at 152.4 107.95)
+		(at 35.56 127)
 		(size 31.75 26.67)
 		(exclude_from_sim no)
@@
 		)
 		(property "Sheetname" "MOTOR_DRIVER_M1"
-			(at 152.4 107.2384 0)
+			(at 35.56 126.2884 0)
 			(show_name no)
 			(do_not_autoplace no)
@@
 		)
 		(property "Sheetfile" "motor_driver_m1.kicad_sch"
-			(at 152.4 135.2046 0)
+			(at 35.56 154.2546 0)
 			(show_name no)
 			(do_not_autoplace no)
@@
 	)
 	(sheet
-		(at 205.74 59.69)
+		(at 78.74 91.44)
 		(size 31.75 26.67)
 		(exclude_from_sim no)
@@
 		)
 		(property "Sheetname" "MOTOR_DRIVER_M4"
-			(at 205.74 58.9784 0)
+			(at 78.74 90.7284 0)
 			(show_name no)
 			(do_not_autoplace no)
@@
 		)
 		(property "Sheetfile" "motor_driver_m4.kicad_sch"
-			(at 205.74 86.9446 0)
+			(at 78.74 118.6946 0)
 			(show_name no)
 			(do_not_autoplace no)
@@
 	)
 	(sheet
-		(at 91.44 109.22)
-		(size 29.21 25.4)
-		(exclude_from_sim no)
-		(in_bom yes)
-		(on_board yes)
-		(dnp no)
-		(fields_autoplaced yes)
-		(stroke
-			(width 0.1524)
-			(type solid)
-		)
-		(fill
-			(color 0 0 0 0)
-		)
-		(property "Sheetname" "GPIO-CONN"
-			(at 91.44 108.5084 0)
-			(show_name no)
-			(do_not_autoplace no)
-			(effects
-				(font
-					(size 1.27 1.27)
-				)
-				(justify left bottom)
-			)
-		)
-		(property "Sheetfile" "gpio-conn.kicad_sch"
-			(at 91.44 135.2046 0)
-			(show_name no)
-			(do_not_autoplace no)
-			(effects
-				(font
-					(size 1.27 1.27)
-				)
-				(justify left top)
-			)
-		)
-		(instances
-			(project "esc"
-				(path "/131092d7-5dad-4272-a758-a2445b6ec99c"
-					(page "3")
-				)
-			)
-		)
-	)
-	(sheet
-		(at 36.83 109.22)
+		(at 35.56 33.02)
 		(size 29.21 22.86)
 		(exclude_from_sim no)
@@
 		)
 		(property "Sheetname" "POWER CONN"
-			(at 36.83 108.5084 0)
+			(at 35.56 32.3084 0)
 			(show_name no)
 			(do_not_autoplace no)
@@
 		)
 		(property "Sheetfile" "power_conn.kicad_sch"
-			(at 36.83 132.6646 0)
+			(at 35.56 56.4646 0)
 			(show_name no)
 			(do_not_autoplace no)
@@
 	)
 	(sheet
-		(at 207.01 107.95)
+		(at 78.74 128.27)
 		(size 31.75 26.67)
 		(exclude_from_sim no)
@@
 		)
 		(property "Sheetname" "MOTOR_DRIVER_M2"
-			(at 207.01 107.2384 0)
+			(at 78.74 127.5584 0)
 			(show_name no)
 			(do_not_autoplace no)
@@
 		)
 		(property "Sheetfile" "motor_driver_m2.kicad_sch"
-			(at 207.01 135.2046 0)
-			(show_name no)
-			(do_not_autoplace no)
+			(at 78.74 155.5246 0)
+			(show_name no)
+			(do_not_autoplace no)
