File: gpio-conn.kicad_sch (KiCad schematic)
At the start: 6 parts, among them J21 Conn_01x01_Pin, J22 Conn_01x01_Pin, J23 Conn_01x01_Pin, J24 Conn_01x01_Pin, J25 Conn_01x01_Pin, J3 Conn_01x01_Pin

Commit message: ...
Parts:
- added J26, J27: Conn_01x01_Pin, deshan:Conn_01x01_Pin, symbol Connector:Conn_01x01_Pin
- J21, J22, J23, J25, J3: footprint deshan:Conn_1x1_small -> deshan:Conn_01x01_Pin
- J24: value Conn_01x01_Pin -> (none); footprint deshan:Conn_1x1_small -> deshan:Conn_01x01_Pin
Connections:
- net SWCLK_H renamed SWCLK_M1
- net SWCLK_L renamed SWCLK_M2
- new net SWCLK_M3: J26.1 (Pin_1)
- new net SWCLK_M4: J27.1 (Pin_1)
Changed lines of the file:
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@@
 	(text_box "ST-LINK-CONN"
 		(exclude_from_sim no)
-		(at 58.42 40.64 0)
+		(at 57.15 43.18 0)
 		(size 53.34 53.34)
 		(margins 0.9525 0.9525 0.9525 0.9525)
@@
 		)
 	)
-	(global_label "SWCLK_H"
+	(global_label "SWCLK_M1"
 		(shape input)
 		(at 77.47 53.34 180)
@@
 		)
 		(property "Intersheetrefs" "${INTERSHEET_REFS}"
-			(at 65.9577 53.34 0)
+			(at 64.6273 53.34 0)
 			(hide yes)
 			(show_name no)
@@
 		)
 	)
-	(global_label "SWCLK_L"
+	(global_label "SWCLK_M2"
 		(shape input)
 		(at 77.47 58.42 180)
@@
 		)
 		(property "Intersheetrefs" "${INTERSHEET_REFS}"
-			(at 66.2601 58.42 0)
+			(at 64.6273 58.42 0)
+			(hide yes)
+			(show_name no)
+			(do_not_autoplace no)
+			(effects
+				(font
+					(size 1.27 1.27)
+				)
+				(justify right)
+			)
+		)
+	)
+	(global_label "SWCLK_M3"
+		(shape input)
+		(at 77.47 63.5 180)
+		(fields_autoplaced yes)
+		(effects
+			(font
+				(size 1.27 1.27)
+			)
+			(justify right)
+		)
+		(property "Intersheetrefs" "${INTERSHEET_REFS}"
+			(at 64.6273 63.5 0)
 			(hide yes)
 			(show_name no)
@@
 		(property "Intersheetrefs" "${INTERSHEET_REFS}"
 			(at 64.9901 87.63 0)
+			(hide yes)
+			(show_name no)
+			(do_not_autoplace no)
+			(effects
+				(font
+					(size 1.27 1.27)
+				)
+				(justify right)
+			)
+		)
+	)
+	(global_label "SWCLK_M4"
+		(shape input)
+		(at 77.47 68.58 180)
+		(fields_autoplaced yes)
+		(effects
+			(font
+				(size 1.27 1.27)
+			)
+			(justify right)
+		)
+		(property "Intersheetrefs" "${INTERSHEET_REFS}"
+			(at 64.6273 68.58 0)
 			(hide yes)
 			(show_name no)
@@
 			)
 		)
-		(property "Footprint" "deshan:Conn_1x1_small"
+		(property "Footprint" "deshan:Conn_01x01_Pin"
 			(at 82.55 78.74 0)
 			(hide yes)
@@
 			)
 		)
-		(property "Value" "Conn_01x01_Pin"
+		(property "Value" ""
 			(at 91.44 83.566 0)
 			(show_name no)
@@
 			)
 		)
-		(property "Footprint" "deshan:Conn_1x1_small"
+		(property "Footprint" "deshan:Conn_01x01_Pin"
 			(at 82.55 83.82 0)
 			(hide yes)
@@
 	(symbol
 		(lib_id "Connector:Conn_01x01_Pin")
+		(at 82.55 68.58 180)
+		(unit 1)
+		(body_style 1)
+		(exclude_from_sim no)
+		(in_bom yes)
+		(on_board yes)
+		(in_pos_files yes)
+		(dnp no)
+		(property "Reference" "J27"
+			(at 82.677 66.548 0)
+			(show_name no)
+			(do_not_autoplace no)
+			(effects
+				(font
+					(size 1.27 1.27)
+				)
+			)
+		)
+		(property "Value" "Conn_01x01_Pin"
+			(at 91.694 68.58 0)
+			(show_name no)
+			(do_not_autoplace no)
+			(effects
+				(font
+					(size 1.27 1.27)
+				)
+			)
+		)
+		(property "Footprint" "deshan:Conn_01x01_Pin"
+			(at 82.55 68.58 0)
+			(hide yes)
+			(show_name no)
+			(do_not_autoplace no)
+			(effects
+				(font
+					(size 1.27 1.27)
+				)
+			)
+		)
+		(property "Datasheet" ""
+			(at 82.55 68.58 0)
+			(hide yes)
+			(show_name no)
+			(do_not_autoplace no)
+			(effects
+				(font
+					(size 1.27 1.27)
+				)
+			)
+		)
+		(property "Description" "Generic connector, single row, 01x01, script generated"
+			(at 82.55 68.58 0)
+			(hide yes)
+			(show_name no)
+			(do_not_autoplace no)
+			(effects
+				(font
+					(size 1.27 1.27)
+				)
+			)
+		)
+		(pin "1"
+		)
+		(instances
+			(project "esc"
+				(path "/131092d7-5dad-4272-a758-a2445b6ec99c/d06f5338-d839-45bd-ae1a-cb9d2da3e16c"
+					(reference "J27")
+					(unit 1)
+				)
+			)
+		)
+	)
+	(symbol
+		(lib_id "Connector:Conn_01x01_Pin")
 		(at 82.55 53.34 180)
 		(unit 1)
@@
 		(dnp no)
 		(property "Reference" "J21"
-			(at 81.915 48.26 0)
+			(at 82.677 51.308 0)
 			(show_name no)
 			(do_not_autoplace no)
@@
 			)
 		)
-		(property "Footprint" "deshan:Conn_1x1_small"
+		(property "Footprint" "deshan:Conn_01x01_Pin"
 			(at 82.55 53.34 0)
 			(hide yes)
@@
 				(path "/131092d7-5dad-4272-a758-a2445b6ec99c/d06f5338-d839-45bd-ae1a-cb9d2da3e16c"
 					(reference "J21")
+					(unit 1)
+				)
+			)
+		)
+	)
+	(symbol
+		(lib_id "Connector:Conn_01x01_Pin")
+		(at 82.55 63.5 180)
+		(unit 1)
+		(body_style 1)
+		(exclude_from_sim no)
+		(in_bom yes)
+		(on_board yes)
+		(in_pos_files yes)
+		(dnp no)
+		(property "Reference" "J26"
+			(at 82.677 61.468 0)
+			(show_name no)
+			(do_not_autoplace no)
+			(effects
+				(font
+					(size 1.27 1.27)
+				)
+			)
+		)
+		(property "Value" "Conn_01x01_Pin"
+			(at 91.694 63.5 0)
+			(show_name no)
+			(do_not_autoplace no)
+			(effects
+				(font
+					(size 1.27 1.27)
+				)
+			)
+		)
+		(property "Footprint" "deshan:Conn_01x01_Pin"
+			(at 82.55 63.5 0)
+			(hide yes)
+			(show_name no)
+			(do_not_autoplace no)
+			(effects
+				(font
+					(size 1.27 1.27)
+				)
+			)
+		)
+		(property "Datasheet" ""
+			(at 82.55 63.5 0)
+			(hide yes)
+			(show_name no)
+			(do_not_autoplace no)
+			(effects
+				(font
+					(size 1.27 1.27)
+				)
+			)
+		)
+		(property "Description" "Generic connector, single row, 01x01, script generated"
+			(at 82.55 63.5 0)
+			(hide yes)
+			(show_name no)
+			(do_not_autoplace no)
+			(effects
+				(font
+					(size 1.27 1.27)
+				)
+			)
+		)
+		(pin "1"
+		)
+		(instances
+			(project "esc"
+				(path "/131092d7-5dad-4272-a758-a2445b6ec99c/d06f5338-d839-45bd-ae1a-cb9d2da3e16c"
+					(reference "J26")
 					(unit 1)
 				)
@@
 			)
 		)
-		(property "Footprint" "deshan:Conn_1x1_small"
+		(property "Footprint" "deshan:Conn_01x01_Pin"
 			(at 82.55 74.93 0)
 			(hide yes)
@@
 			)
 		)
-		(property "Footprint" "deshan:Conn_1x1_small"
+		(property "Footprint" "deshan:Conn_01x01_Pin"
 			(at 82.55 87.63 0)
 			(hide yes)
@@
 			)
 		)
-		(property "Footprint" "deshan:Conn_1x1_small"
+		(property "Footprint" "deshan:Conn_01x01_Pin"
 			(at 82.55 58.42 0)
 			(hide yes)

Commit message: ...
Parts:
- renumbered J21 to SWCLK_M1, J23 to SWCLK_M2, J26 to SWCLK_M3, J27 to SWCLK_M4, J3 to SWDIO_M1, J22 to SWDIO_M2, J24 to SWDIO_M3, J25 to SWDIO_M4
Other:
- moved on the sheet: SWDIO_M2, SWDIO_M4
Changed lines of the file:
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@@
 	(global_label "SWDIO_M4"
 		(shape input)
-		(at 77.47 87.63 180)
+		(at 77.47 88.9 180)
 		(fields_autoplaced yes)
 		(effects
@@
 		)
 		(property "Intersheetrefs" "${INTERSHEET_REFS}"
-			(at 64.9901 87.63 0)
+			(at 64.9901 88.9 0)
 			(hide yes)
 			(show_name no)
@@
 	(global_label "SWDIO_M2"
 		(shape input)
-		(at 77.47 78.74 180)
+		(at 77.47 80.01 180)
 		(fields_autoplaced yes)
 		(effects
@@
 		)
 		(property "Intersheetrefs" "${INTERSHEET_REFS}"
-			(at 64.9901 78.74 0)
+			(at 64.9901 80.01 0)
 			(hide yes)
 			(show_name no)
@@
 	(symbol
 		(lib_id "Connector:Conn_01x01_Pin")
-		(at 82.55 78.74 180)
-		(unit 1)
-		(body_style 1)
-		(exclude_from_sim no)
-		(in_bom yes)
-		(on_board yes)
-		(in_pos_files yes)
-		(dnp no)
-		(property "Reference" "J22"
-			(at 82.423 77.216 0)
+		(at 82.55 80.01 180)
+		(unit 1)
+		(body_style 1)
+		(exclude_from_sim no)
+		(in_bom yes)
+		(on_board yes)
+		(in_pos_files yes)
+		(dnp no)
+		(property "Reference" "SWDIO_M2"
+			(at 88.265 78.232 0)
 			(show_name no)
 			(do_not_autoplace no)
@@
 		)
 		(property "Value" "Conn_01x01_Pin"
-			(at 91.44 78.74 0)
-			(show_name no)
-			(do_not_autoplace no)
-			(effects
-				(font
-					(size 1.27 1.27)
-				)
-			)
-		)
-		(property "Footprint" "deshan:Conn_01x01_Pin"
-			(at 82.55 78.74 0)
-			(hide yes)
-			(show_name no)
-			(do_not_autoplace no)
-			(effects
-				(font
-					(size 1.27 1.27)
-				)
-			)
-		)
-		(property "Datasheet" ""
-			(at 82.55 78.74 0)
-			(hide yes)
-			(show_name no)
-			(do_not_autoplace no)
-			(effects
-				(font
-					(size 1.27 1.27)
-				)
-			)
-		)
-		(property "Description" "Generic connector, single row, 01x01, script generated"
-			(at 82.55 78.74 0)
-			(hide yes)
-			(show_name no)
-			(do_not_autoplace no)
-			(effects
-				(font
-					(size 1.27 1.27)
-				)
-			)
-		)
-		(pin "1"
-		)
-		(instances
-			(project "esc"
-				(path "/131092d7-5dad-4272-a758-a2445b6ec99c/d06f5338-d839-45bd-ae1a-cb9d2da3e16c"
-					(reference "J22")
+			(at 91.44 80.01 0)
+			(show_name no)
+			(do_not_autoplace no)
+			(effects
+				(font
+					(size 1.27 1.27)
+				)
+			)
+		)
+		(property "Footprint" "deshan:Conn_01x01_Pin"
+			(at 82.55 80.01 0)
+			(hide yes)
+			(show_name no)
+			(do_not_autoplace no)
+			(effects
+				(font
+					(size 1.27 1.27)
+				)
+			)
+		)
+		(property "Datasheet" ""
+			(at 82.55 80.01 0)
+			(hide yes)
+			(show_name no)
+			(do_not_autoplace no)
+			(effects
+				(font
+					(size 1.27 1.27)
+				)
+			)
+		)
+		(property "Description" "Generic connector, single row, 01x01, script generated"
+			(at 82.55 80.01 0)
+			(hide yes)
+			(show_name no)
+			(do_not_autoplace no)
+			(effects
+				(font
+					(size 1.27 1.27)
+				)
+			)
+		)
+		(pin "1"
+		)
+		(instances
+			(project "esc"
+				(path "/131092d7-5dad-4272-a758-a2445b6ec99c/d06f5338-d839-45bd-ae1a-cb9d2da3e16c"
+					(reference "SWDIO_M2")
 					(unit 1)
 				)
@@
 		(in_pos_files yes)
 		(dnp no)
-		(property "Reference" "J24"
-			(at 82.423 82.042 0)
+		(property "Reference" "SWDIO_M3"
+			(at 88.265 83.312 0)
 			(show_name no)
 			(do_not_autoplace no)
@@
 			(project "esc"
 				(path "/131092d7-5dad-4272-a758-a2445b6ec99c/d06f5338-d839-45bd-ae1a-cb9d2da3e16c"
-					(reference "J24")
+					(reference "SWDIO_M3")
 					(unit 1)
 				)
@@
 		(in_pos_files yes)
 		(dnp no)
-		(property "Reference" "J27"
-			(at 82.677 66.548 0)
+		(property "Reference" "SWCLK_M4"
+			(at 88.519 66.548 0)
 			(show_name no)
 			(do_not_autoplace no)
@@
 			(project "esc"
 				(path "/131092d7-5dad-4272-a758-a2445b6ec99c/d06f5338-d839-45bd-ae1a-cb9d2da3e16c"
-					(reference "J27")
+					(reference "SWCLK_M4")
 					(unit 1)
 				)
@@
 		(in_pos_files yes)
 		(dnp no)
-		(property "Reference" "J21"
-			(at 82.677 51.308 0)
+		(property "Reference" "SWCLK_M1"
+			(at 88.773 51.562 0)
 			(show_name no)
 			(do_not_autoplace no)
@@
 			(project "esc"
 				(path "/131092d7-5dad-4272-a758-a2445b6ec99c/d06f5338-d839-45bd-ae1a-cb9d2da3e16c"
-					(reference "J21")
+					(reference "SWCLK_M1")
 					(unit 1)
 				)
@@
 		(in_pos_files yes)
 		(dnp no)
-		(property "Reference" "J26"
-			(at 82.677 61.468 0)
+		(property "Reference" "SWCLK_M3"
+			(at 88.773 61.722 0)
 			(show_name no)
 			(do_not_autoplace no)
@@
 			(project "esc"
 				(path "/131092d7-5dad-4272-a758-a2445b6ec99c/d06f5338-d839-45bd-ae1a-cb9d2da3e16c"
-					(reference "J26")
+					(reference "SWCLK_M3")
 					(unit 1)
 				)
@@
 		(in_pos_files yes)
 		(dnp no)
-		(property "Reference" "J3"
-			(at 82.423 73.152 0)
+		(property "Reference" "SWDIO_M1"
+			(at 88.011 72.898 0)
 			(show_name no)
 			(do_not_autoplace no)
@@
 			(project "esc"
 				(path "/131092d7-5dad-4272-a758-a2445b6ec99c/d06f5338-d839-45bd-ae1a-cb9d2da3e16c"
-					(reference "J3")
-					(unit 1)
-				)
-			)
-		)
-	)
-	(symbol
-		(lib_id "Connector:Conn_01x01_Pin")
-		(at 82.55 87.63 180)
-		(unit 1)
-		(body_style 1)
-		(exclude_from_sim no)
-		(in_bom yes)
-		(on_board yes)
-		(in_pos_files yes)
-		(dnp no)
-		(property "Reference" "J25"
-			(at 82.423 86.106 0)
+					(reference "SWDIO_M1")
+					(unit 1)
+				)
+			)
+		)
+	)
+	(symbol
+		(lib_id "Connector:Conn_01x01_Pin")
+		(at 82.55 88.9 180)
+		(unit 1)
+		(body_style 1)
+		(exclude_from_sim no)
+		(in_bom yes)
+		(on_board yes)
+		(in_pos_files yes)
+		(dnp no)
+		(property "Reference" "SWDIO_M4"
+			(at 88.265 86.868 0)
 			(show_name no)
 			(do_not_autoplace no)
@@
 		)
 		(property "Value" "Conn_01x01_Pin"
-			(at 91.44 87.63 0)
-			(show_name no)
-			(do_not_autoplace no)
-			(effects
-				(font
-					(size 1.27 1.27)
-				)
-			)
-		)
-		(property "Footprint" "deshan:Conn_01x01_Pin"
-			(at 82.55 87.63 0)
-			(hide yes)
-			(show_name no)
-			(do_not_autoplace no)
-			(effects
-				(font
-					(size 1.27 1.27)
-				)
-			)
-		)
-		(property "Datasheet" ""
-			(at 82.55 87.63 0)
-			(hide yes)
-			(show_name no)
-			(do_not_autoplace no)
-			(effects
-				(font
-					(size 1.27 1.27)
-				)
-			)
-		)
-		(property "Description" "Generic connector, single row, 01x01, script generated"
-			(at 82.55 87.63 0)
-			(hide yes)
-			(show_name no)
-			(do_not_autoplace no)
-			(effects
-				(font
-					(size 1.27 1.27)
-				)
-			)
-		)
-		(pin "1"
-		)
-		(instances
-			(project "esc"
-				(path "/131092d7-5dad-4272-a758-a2445b6ec99c/d06f5338-d839-45bd-ae1a-cb9d2da3e16c"
-					(reference "J25")
+			(at 91.44 88.9 0)
+			(show_name no)
+			(do_not_autoplace no)
+			(effects
+				(font
+					(size 1.27 1.27)
+				)
+			)
+		)
+		(property "Footprint" "deshan:Conn_01x01_Pin"
+			(at 82.55 88.9 0)
+			(hide yes)
+			(show_name no)
+			(do_not_autoplace no)
+			(effects
+				(font
+					(size 1.27 1.27)
+				)
+			)
+		)
+		(property "Datasheet" ""
+			(at 82.55 88.9 0)
+			(hide yes)
+			(show_name no)
+			(do_not_autoplace no)
+			(effects
+				(font
+					(size 1.27 1.27)
+				)
+			)
+		)
+		(property "Description" "Generic connector, single row, 01x01, script generated"
+			(at 82.55 88.9 0)
+			(hide yes)
+			(show_name no)
+			(do_not_autoplace no)
+			(effects
+				(font
+					(size 1.27 1.27)
+				)
+			)
+		)
+		(pin "1"
+		)
+		(instances
+			(project "esc"
+				(path "/131092d7-5dad-4272-a758-a2445b6ec99c/d06f5338-d839-45bd-ae1a-cb9d2da3e16c"
+					(reference "SWDIO_M4")
 					(unit 1)
 				)
@@
 		(in_pos_files yes)
 		(dnp no)
-		(property "Reference" "J23"
-			(at 82.677 56.388 0)
+		(property "Reference" "SWCLK_M2"
+			(at 89.027 56.388 0)
 			(show_name no)
 			(do_not_autoplace no)
@@
 			(project "esc"
 				(path "/131092d7-5dad-4272-a758-a2445b6ec99c/d06f5338-d839-45bd-ae1a-cb9d2da3e16c"
-					(reference "J23")
-					(unit 1)
-				)
+					(reference "SWCLK_M2")
+					(unit 1)
+				)

Commit message: ...
Parts:
- removed SWCLK_M1, SWCLK_M2, SWCLK_M3, SWCLK_M4, SWDIO_M1, SWDIO_M2, SWDIO_M4: Conn_01x01_Pin, deshan:Conn_01x01_Pin, symbol Connector:Conn_01x01_Pin
- removed SWDIO_M3: (no value), deshan:Conn_01x01_Pin, symbol Connector:Conn_01x01_Pin
