File: motor_driver_m2.kicad_sch (KiCad schematic)
At the start: 50 parts, among them J4 Conn_01x01_Pin, J5 Conn_01x01_Pin, J6 Conn_01x01_Pin, M2 STM32C011F6U6TR, Q10 NP80N06D6, Q11 NP80N06D6, Q12 NP80N06D6, Q7 NP80N06D6, Q8 NP80N06D6, Q9 NP80N06D6

Commit message: ...
Parts:
- added SWCLK_M2, SWDIO_M2: Conn_01x01_Pin, deshan:Conn_01x01_Pin, symbol Connector:Conn_01x01_Pin
- R20: value 18k -> 100k
- R21: value 10k -> 18k
Connections:
- net SWCLK_M2: now also SWCLK_M2.1 (Pin_1)
- net SWDIO_M2: now also SWDIO_M2.1 (Pin_1)
Other:
- moved on the sheet: C16, C17, C18, C19, C20, C21, C22, C23, C24, C25, C26, C27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
