File: motor_driver_m2.kicad_sch (KiCad schematic)
At the start: 52 parts, among them J4 Conn_01x01_Pin, J5 Conn_01x01_Pin, J6 Conn_01x01_Pin, M2 STM32C011F6U6TR, Q10 NP80N06D6, Q11 NP80N06D6, Q12 NP80N06D6, Q7 NP80N06D6, Q8 NP80N06D6, Q9 NP80N06D6

Commit message: ...
Parts:
- C25, C26, C27: footprint easyeda2kicad:C0603 -> easyeda2kicad:C1206
Changed lines of the file:
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@@
 			)
 		)
-		(property "Footprint" "easyeda2kicad:C0603"
+		(property "Footprint" "easyeda2kicad:C1206"
 			(at 270.2052 140.97 0)
 			(hide yes)
@@
 			)
 		)
-		(property "Footprint" "easyeda2kicad:C0603"
+		(property "Footprint" "easyeda2kicad:C1206"
 			(at 268.9352 46.99 0)
 			(hide yes)
@@
 			)
 		)
-		(property "Footprint" "easyeda2kicad:C0603"
+		(property "Footprint" "easyeda2kicad:C1206"
 			(at 270.2052 93.98 0)
 			(hide yes)
