File: motor_driver_m3.kicad_sch (KiCad schematic)
At the start: 52 parts, among them J7 Conn_01x01_Pin, J8 Conn_01x01_Pin, J9 Conn_01x01_Pin, M3 STM32C011F6U6TR, Q13 NP80N06D6, Q14 NP80N06D6, Q15 NP80N06D6, Q16 NP80N06D6, Q17 NP80N06D6, Q18 NP80N06D6

Commit message: ...
Parts:
- C40, C41, C42: footprint easyeda2kicad:C0603 -> easyeda2kicad:C1206
Changed lines of the file:
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@@
 			)
 		)
-		(property "Footprint" "easyeda2kicad:C0603"
+		(property "Footprint" "easyeda2kicad:C1206"
 			(at 274.0152 46.99 0)
 			(hide yes)
@@
 			)
 		)
-		(property "Footprint" "easyeda2kicad:C0603"
+		(property "Footprint" "easyeda2kicad:C1206"
 			(at 274.0152 93.98 0)
 			(hide yes)
@@
 			)
 		)
-		(property "Footprint" "easyeda2kicad:C0603"
+		(property "Footprint" "easyeda2kicad:C1206"
 			(at 274.0152 143.51 0)
 			(hide yes)
