File: motor_driver_m4.kicad_sch (KiCad schematic)
At the start: 50 parts, among them J10 Conn_01x01_Pin, J11 Conn_01x01_Pin, J12 Conn_01x01_Pin, M4 STM32C011F6U6TR, Q19 NP80N06D6, Q20 NP80N06D6, Q21 NP80N06D6, Q22 NP80N06D6, Q23 NP80N06D6, Q24 NP80N06D6

Commit message: ...
Parts:
- added SWCLK_M4, SWDIO_M4: Conn_01x01_Pin, deshan:Conn_01x01_Pin, symbol Connector:Conn_01x01_Pin
- R56: value 18k -> 100k
- R57: value 10k -> 18k
Connections:
- net SWCLK_M4: now also SWCLK_M4.1 (Pin_1)
- net SWDIO_M4: now also SWDIO_M4.1 (Pin_1)
Other:
- moved on the sheet: C46, C47, C48, C49, C50, C51, C52, C53, C54, C55, C56, C57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
