File: motor_driver_m4.kicad_sch (KiCad schematic)
At the start: 52 parts, among them J10 Conn_01x01_Pin, J11 Conn_01x01_Pin, J12 Conn_01x01_Pin, M4 STM32C011F6U6TR, Q19 NP80N06D6, Q20 NP80N06D6, Q21 NP80N06D6, Q22 NP80N06D6, Q23 NP80N06D6, Q24 NP80N06D6

Commit message: ...
Parts:
- C55, C56, C57: footprint easyeda2kicad:C0603 -> easyeda2kicad:C1206
Changed lines of the file:
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@@
 			)
 		)
-		(property "Footprint" "easyeda2kicad:C0603"
+		(property "Footprint" "easyeda2kicad:C1206"
 			(at 271.4752 142.24 0)
 			(hide yes)
@@
 			)
 		)
-		(property "Footprint" "easyeda2kicad:C0603"
+		(property "Footprint" "easyeda2kicad:C1206"
 			(at 270.2052 46.99 0)
 			(hide yes)
@@
 			)
 		)
-		(property "Footprint" "easyeda2kicad:C0603"
+		(property "Footprint" "easyeda2kicad:C1206"
 			(at 270.2052 93.98 0)
 			(hide yes)
