File: power_conn.kicad_sch (KiCad schematic)
At the start: 11 parts, among them J1 Conn_01x02, U1 AP63201WU-7

Commit message: ...
Parts:
- renumbered C2 to C0, C3 to C2, C4 to C3, C2.1 to C4, C2.2 to C5, R2 to R1, R1 to R2
Changed lines of the file:
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@@
 		(dnp no)
 		(fields_autoplaced yes)
-		(property "Reference" "C4"
+		(property "Reference" "C3"
 			(at 163.83 54.6099 0)
 			(effects
@@
 			(project "esc"
 				(path "/131092d7-5dad-4272-a758-a2445b6ec99c/d16f723d-eb96-498f-9f42-02a776bee3f3"
-					(reference "C4")
+					(reference "C3")
 					(unit 1)
 				)
@@
 		(dnp no)
 		(fields_autoplaced yes)
-		(property "Reference" "#PWR014"
+		(property "Reference" "#PWR05"
 			(at 179.07 87.63 0)
 			(effects
@@
 			(project "esc"
 				(path "/131092d7-5dad-4272-a758-a2445b6ec99c/d16f723d-eb96-498f-9f42-02a776bee3f3"
-					(reference "#PWR014")
+					(reference "#PWR05")
 					(unit 1)
 				)
@@
 		(dnp no)
 		(fields_autoplaced yes)
-		(property "Reference" "#FLG02"
+		(property "Reference" "#FLG03"
 			(at 195.58 64.135 0)
 			(effects
@@
 			(project "esc"
 				(path "/131092d7-5dad-4272-a758-a2445b6ec99c/d16f723d-eb96-498f-9f42-02a776bee3f3"
-					(reference "#FLG02")
+					(reference "#FLG03")
 					(unit 1)
 				)
@@
 		(dnp no)
 		(fields_autoplaced yes)
-		(property "Reference" "#FLG04"
+		(property "Reference" "#FLG02"
 			(at 39.37 43.815 0)
 			(effects
@@
 			(project "esc"
 				(path "/131092d7-5dad-4272-a758-a2445b6ec99c/d16f723d-eb96-498f-9f42-02a776bee3f3"
-					(reference "#FLG04")
+					(reference "#FLG02")
 					(unit 1)
 				)
@@
 		(dnp no)
 		(fields_autoplaced yes)
-		(property "Reference" "C2.1"
+		(property "Reference" "C4"
 			(at 182.88 71.1199 0)
 			(effects
@@
 			(project "esc"
 				(path "/131092d7-5dad-4272-a758-a2445b6ec99c/d16f723d-eb96-498f-9f42-02a776bee3f3"
-					(reference "C2.1")
+					(reference "C4")
 					(unit 1)
 				)
@@
 		(dnp no)
 		(fields_autoplaced yes)
-		(property "Reference" "C2"
+		(property "Reference" "C0"
 			(at 54.61 38.0999 90)
 			(effects
@@
 			(project ""
 				(path "/131092d7-5dad-4272-a758-a2445b6ec99c/d16f723d-eb96-498f-9f42-02a776bee3f3"
-					(reference "C2")
+					(reference "C0")
 					(unit 1)
 				)
@@
 		(on_board yes)
 		(dnp no)
-		(property "Reference" "#PWR015"
+		(property "Reference" "#PWR01"
 			(at 30.48 41.91 0)
 			(effects
@@
 			(project "esc"
 				(path "/131092d7-5dad-4272-a758-a2445b6ec99c/d16f723d-eb96-498f-9f42-02a776bee3f3"
-					(reference "#PWR015")
+					(reference "#PWR01")
 					(unit 1)
 				)
@@
 		(dnp no)
 		(fields_autoplaced yes)
-		(property "Reference" "C3"
+		(property "Reference" "C2"
 			(at 139.7 53.34 90)
 			(effects
@@
 			(project "esc"
 				(path "/131092d7-5dad-4272-a758-a2445b6ec99c/d16f723d-eb96-498f-9f42-02a776bee3f3"
-					(reference "C3")
+					(reference "C2")
 					(unit 1)
 				)
@@
 		(dnp no)
 		(fields_autoplaced yes)
-		(property "Reference" "C2.2"
+		(property "Reference" "C5"
 			(at 194.31 71.1199 0)
 			(effects
@@
 			(project "esc"
 				(path "/131092d7-5dad-4272-a758-a2445b6ec99c/d16f723d-eb96-498f-9f42-02a776bee3f3"
-					(reference "C2.2")
+					(reference "C5")
 					(unit 1)
 				)
@@
 		(on_board yes)
 		(dnp no)
-		(property "Reference" "R2"
+		(property "Reference" "R1"
 			(at 178.562 39.37 0)
 			(effects
@@
 			(project "esc"
 				(path "/131092d7-5dad-4272-a758-a2445b6ec99c/d16f723d-eb96-498f-9f42-02a776bee3f3"
-					(reference "R2")
+					(reference "R1")
 					(unit 1)
 				)
@@
 		(on_board yes)
 		(dnp no)
-		(property "Reference" "R1"
+		(property "Reference" "R2"
 			(at 178.562 54.61 0)
 			(effects
@@
 			(project "esc"
 				(path "/131092d7-5dad-4272-a758-a2445b6ec99c/d16f723d-eb96-498f-9f42-02a776bee3f3"
-					(reference "R1")
+					(reference "R2")
 					(unit 1)
 				)
@@
 		(dnp no)
 		(fields_autoplaced yes)
-		(property "Reference" "#PWR05"
+		(property "Reference" "#PWR04"
 			(at 172.72 29.21 0)
 			(effects
@@
 			(project "esc"
 				(path "/131092d7-5dad-4272-a758-a2445b6ec99c/d16f723d-eb96-498f-9f42-02a776bee3f3"
-					(reference "#PWR05")
-					(unit 1)
-				)
+					(reference "#PWR04")
+					(unit 1)
+				)

Commit message: ESC_V1.0
Parts:
- added J16: Conn_01x02, deshan:Batt_Conn_HV, symbol Connector_Generic:Conn_01x02
- added J17: Conn_01x01_Pin, deshan:Conn_1x1_small, symbol Connector:Conn_01x01_Pin
Connections:
- net 3V3: now also J17.1 (Pin_1)
- net B+: now also J16.1 (Pin_1)
- net GND: now also J16.2 (Pin_2)

Commit message: ...
Other:
- title: (none) -> POWER CONNECTORS
Changed lines of the file:
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@@
 	(generator_version "10.0")
 	(paper "A4")
+	(title_block
+		(title "POWER CONNECTORS")
+		(rev "1.0")
+	)
 	(text_box "VOLTAGE-REGULATOR-(OPTIONAL)\n"
 		(exclude_from_sim no)

Commit message: ...
Parts:
- renumbered C1 to CX1, C2 to CX2, C3 to CX3, C4 to CX4, C5 to CX5, L1 to LX1, R1 to RX1, R2 to RX2, U1 to UX1
Changed lines of the file:
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@@
 		(dnp no)
 		(fields_autoplaced yes)
-		(property "Reference" "C3"
+		(property "Reference" "CX3"
 			(at 163.83 54.6099 0)
 			(show_name no)
@@
 			(project "esc"
 				(path "/131092d7-5dad-4272-a758-a2445b6ec99c/d16f723d-eb96-498f-9f42-02a776bee3f3"
-					(reference "C3")
+					(reference "CX3")
 					(unit 1)
 				)
@@
 		(dnp no)
 		(fields_autoplaced yes)
-		(property "Reference" "U1"
+		(property "Reference" "UX1"
 			(at 124.46 55.88 0)
 			(show_name no)
@@
 			(project "esc"
 				(path "/131092d7-5dad-4272-a758-a2445b6ec99c/d16f723d-eb96-498f-9f42-02a776bee3f3"
-					(reference "U1")
+					(reference "UX1")
 					(unit 1)
 				)
@@
 		(dnp no)
 		(fields_autoplaced yes)
-		(property "Reference" "C1"
+		(property "Reference" "CX1"
 			(at 111.76 73.6599 0)
 			(show_name no)
@@
 			(project "esc"
 				(path "/131092d7-5dad-4272-a758-a2445b6ec99c/d16f723d-eb96-498f-9f42-02a776bee3f3"
-					(reference "C1")
+					(reference "CX1")
 					(unit 1)
 				)
@@
 		(dnp no)
 		(fields_autoplaced yes)
-		(property "Reference" "L1"
+		(property "Reference" "LX1"
 			(at 151.13 59.69 0)
 			(show_name no)
@@
 			(project "esc"
 				(path "/131092d7-5dad-4272-a758-a2445b6ec99c/d16f723d-eb96-498f-9f42-02a776bee3f3"
-					(reference "L1")
+					(reference "LX1")
 					(unit 1)
 				)
@@
 		(dnp no)
 		(fields_autoplaced yes)
-		(property "Reference" "C4"
+		(property "Reference" "CX4"
 			(at 182.88 71.1199 0)
 			(show_name no)
@@
 			(project "esc"
 				(path "/131092d7-5dad-4272-a758-a2445b6ec99c/d16f723d-eb96-498f-9f42-02a776bee3f3"
-					(reference "C4")
+					(reference "CX4")
 					(unit 1)
 				)
@@
 		(dnp no)
 		(fields_autoplaced yes)
-		(property "Reference" "C2"
+		(property "Reference" "CX2"
 			(at 139.7 53.34 90)
 			(show_name no)
@@
 			(project "esc"
 				(path "/131092d7-5dad-4272-a758-a2445b6ec99c/d16f723d-eb96-498f-9f42-02a776bee3f3"
-					(reference "C2")
+					(reference "CX2")
 					(unit 1)
 				)
@@
 		(dnp no)
 		(fields_autoplaced yes)
-		(property "Reference" "C5"
+		(property "Reference" "CX5"
 			(at 194.31 71.1199 0)
 			(show_name no)
@@
 			(project "esc"
 				(path "/131092d7-5dad-4272-a758-a2445b6ec99c/d16f723d-eb96-498f-9f42-02a776bee3f3"
-					(reference "C5")
+					(reference "CX5")
 					(unit 1)
 				)
@@
 		(in_pos_files yes)
 		(dnp no)
-		(property "Reference" "R1"
+		(property "Reference" "RX1"
 			(at 178.562 39.37 0)
 			(show_name no)
@@
 			(project "esc"
 				(path "/131092d7-5dad-4272-a758-a2445b6ec99c/d16f723d-eb96-498f-9f42-02a776bee3f3"
-					(reference "R1")
+					(reference "RX1")
 					(unit 1)
 				)
@@
 		(in_pos_files yes)
 		(dnp no)
-		(property "Reference" "R2"
+		(property "Reference" "RX2"
 			(at 178.562 54.61 0)
 			(show_name no)
@@
 			(project "esc"
 				(path "/131092d7-5dad-4272-a758-a2445b6ec99c/d16f723d-eb96-498f-9f42-02a776bee3f3"
-					(reference "R2")
-					(unit 1)
-				)
+					(reference "RX2")
+					(unit 1)
+				)

Commit message: ...
Parts:
- 3V3: renamed from J17; footprint deshan:Conn_1x1_small -> deshan:Conn_01x01_Pin
- POWER_IN1: renamed from J1; footprint deshan:Batt_Conn_HV -> deshan:Conn_01x01_power_x2
- POWER_OUT1: renamed from J16; footprint deshan:Batt_Conn_HV -> deshan:Conn_01x01_power_x2
Changed lines of the file:
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@@
 		(dnp no)
 		(fields_autoplaced yes)
-		(property "Reference" "J1"
+		(property "Reference" "POWER_IN1"
 			(at 68.58 39.3699 0)
 			(show_name no)
@@
 			)
 		)
-		(property "Footprint" "deshan:Batt_Conn_HV"
+		(property "Footprint" "deshan:Conn_01x01_power_x2"
 			(at 66.04 39.37 0)
 			(hide yes)
@@
 			(project "esc"
 				(path "/131092d7-5dad-4272-a758-a2445b6ec99c/d16f723d-eb96-498f-9f42-02a776bee3f3"
-					(reference "J1")
+					(reference "POWER_IN1")
 					(unit 1)
 				)
@@
 		(dnp no)
 		(fields_autoplaced yes)
-		(property "Reference" "J16"
+		(property "Reference" "POWER_OUT1"
 			(at 53.34 59.6899 0)
 			(show_name no)
@@
 			)
 		)
-		(property "Footprint" "deshan:Batt_Conn_HV"
+		(property "Footprint" "deshan:Conn_01x01_power_x2"
 			(at 50.8 59.69 0)
 			(hide yes)
@@
 			(project "esc"
 				(path "/131092d7-5dad-4272-a758-a2445b6ec99c/d16f723d-eb96-498f-9f42-02a776bee3f3"
-					(reference "J16")
+					(reference "POWER_OUT1")
 					(unit 1)
 				)
@@
 		(in_pos_files yes)
 		(dnp no)
-		(fields_autoplaced yes)
-		(property "Reference" "J17"
-			(at 50.165 71.12 0)
+		(property "Reference" "3V3"
+			(at 54.737 73.914 0)
 			(show_name no)
 			(do_not_autoplace no)
@@
 		)
 		(property "Value" "Conn_01x01_Pin"
-			(at 50.165 73.66 0)
-			(show_name no)
-			(do_not_autoplace no)
-			(effects
-				(font
-					(size 1.27 1.27)
-				)
-			)
-		)
-		(property "Footprint" "deshan:Conn_1x1_small"
+			(at 60.579 76.2 0)
+			(show_name no)
+			(do_not_autoplace no)
+			(effects
+				(font
+					(size 1.27 1.27)
+				)
+			)
+		)
+		(property "Footprint" "deshan:Conn_01x01_Pin"
 			(at 50.8 76.2 0)
 			(hide yes)
@@
 			(project "esc"
 				(path "/131092d7-5dad-4272-a758-a2445b6ec99c/d16f723d-eb96-498f-9f42-02a776bee3f3"
-					(reference "J17")
-					(unit 1)
-				)
+					(reference "3V3")
+					(unit 1)
+				)

Commit message: ...
Parts:
- CX1, CX2, CX3, CX4, CX5, LX1, RX1, RX2, UX1: now not fitted; now left out of the parts list
Other:
- note added: "Physical Input connectors for power planes and various power supplies. B+ = Battery +. There is an option to place an internal 3v3 buck regulator to power the board but it is disabled as it cannot fit the current design specifications."
Changed lines of the file:
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@@
 		(title "POWER CONNECTORS")
 		(rev "1.0")
+		(comment 7 "B+ = Battery + ")
+	)
+	(text "Physical Input connectors for power planes and various power supplies.\nB+ = Battery +.\nThere is an option to place an internal 3v3 buck regulator to power the board \nbut it is disabled as it cannot fit the current design specifications."
+		(exclude_from_sim no)
+		(at 177.8 171.196 0)
+		(effects
+			(font
+				(size 1.27 1.27)
+			)
+			(justify left)
+		)
 	)
 	(text_box "VOLTAGE-REGULATOR-(OPTIONAL)\n"
@@
 		(body_style 1)
 		(exclude_from_sim no)
-		(in_bom yes)
-		(on_board yes)
+		(in_bom no)
+		(on_board no)
 		(in_pos_files yes)
-		(dnp no)
+		(dnp yes)
 		(fields_autoplaced yes)
 		(property "Reference" "#PWR06"
@@
 		(body_style 1)
 		(exclude_from_sim no)
-		(in_bom yes)
+		(in_bom no)
 		(on_board no)
 		(in_pos_files yes)
-		(dnp no)
+		(dnp yes)
 		(fields_autoplaced yes)
 		(property "Reference" "CX3"
@@
 		(body_style 1)
 		(exclude_from_sim no)
-		(in_bom yes)
+		(in_bom no)
 		(on_board no)
 		(in_pos_files yes)
-		(dnp no)
+		(dnp yes)
 		(fields_autoplaced yes)
 		(property "Reference" "UX1"
@@
 		(body_style 1)
 		(exclude_from_sim no)
-		(in_bom yes)
-		(on_board yes)
+		(in_bom no)
+		(on_board no)
 		(in_pos_files yes)
-		(dnp no)
+		(dnp yes)
 		(fields_autoplaced yes)
 		(property "Reference" "#PWR05"
@@
 		(body_style 1)
 		(exclude_from_sim no)
-		(in_bom yes)
-		(on_board yes)
+		(in_bom no)
+		(on_board no)
 		(in_pos_files yes)
-		(dnp no)
+		(dnp yes)
 		(fields_autoplaced yes)
 		(property "Reference" "#FLG03"
@@
 		(body_style 1)
 		(exclude_from_sim no)
-		(in_bom yes)
+		(in_bom no)
 		(on_board no)
 		(in_pos_files yes)
-		(dnp no)
+		(dnp yes)
 		(fields_autoplaced yes)
 		(property "Reference" "CX1"
@@
 		(body_style 1)
 		(exclude_from_sim no)
-		(in_bom yes)
+		(in_bom no)
 		(on_board no)
 		(in_pos_files yes)
-		(dnp no)
+		(dnp yes)
 		(fields_autoplaced yes)
 		(property "Reference" "LX1"
@@
 		(body_style 1)
 		(exclude_from_sim no)
-		(in_bom yes)
+		(in_bom no)
 		(on_board no)
 		(in_pos_files yes)
-		(dnp no)
+		(dnp yes)
 		(fields_autoplaced yes)
 		(property "Reference" "CX4"
@@
 		(body_style 1)
 		(exclude_from_sim no)
-		(in_bom yes)
-		(on_board yes)
+		(in_bom no)
+		(on_board no)
 		(in_pos_files yes)
-		(dnp no)
+		(dnp yes)
 		(fields_autoplaced yes)
 		(property "Reference" "#PWR02"
@@
 		(body_style 1)
 		(exclude_from_sim no)
-		(in_bom yes)
-		(on_board yes)
+		(in_bom no)
+		(on_board no)
 		(in_pos_files yes)
-		(dnp no)
+		(dnp yes)
 		(fields_autoplaced yes)
 		(property "Reference" "#PWR03"
@@
 		(body_style 1)
 		(exclude_from_sim no)
-		(in_bom yes)
+		(in_bom no)
 		(on_board no)
 		(in_pos_files yes)
-		(dnp no)
+		(dnp yes)
 		(fields_autoplaced yes)
 		(property "Reference" "CX2"
@@
 		(body_style 1)
 		(exclude_from_sim no)
-		(in_bom yes)
+		(in_bom no)
 		(on_board no)
 		(in_pos_files yes)
-		(dnp no)
+		(dnp yes)
 		(fields_autoplaced yes)
 		(property "Reference" "CX5"
@@
 		(body_style 1)
 		(exclude_from_sim no)
-		(in_bom yes)
+		(in_bom no)
 		(on_board no)
 		(in_pos_files yes)
-		(dnp no)
+		(dnp yes)
 		(property "Reference" "RX1"
 			(at 178.562 39.37 0)
@@
 		(body_style 1)
 		(exclude_from_sim no)
-		(in_bom yes)
+		(in_bom no)
 		(on_board no)
 		(in_pos_files yes)
-		(dnp no)
+		(dnp yes)
 		(property "Reference" "RX2"
 			(at 178.562 54.61 0)
@@
 		(body_style 1)
 		(exclude_from_sim no)
-		(in_bom yes)
-		(on_board yes)
+		(in_bom no)
+		(on_board no)
 		(in_pos_files yes)
-		(dnp no)
+		(dnp yes)
 		(fields_autoplaced yes)
 		(property "Reference" "#PWR04"
